Commit message: ..

File: src/lbr_fri_ros2_stack/lbr_description/urdf/dual_iiwa7/dual_iiwa7_mod.urdf (robot description, URDF)
Before this commit: robot dual_iiwa7, 19 links, 18 joints
Joints:
- joint world_kuka_blue_joint: origin xyz=0 0 0 rpy=0 0 0 -> xyz=0.7 -0.3 0 rpy=0 0 0
- joint world_kuka_green_joint: origin xyz=1 1 0 rpy=0 0 0 -> xyz=0.75 0.9 0 rpy=0 0 0

Commit message: fixed all cartesian planner and added stop flag for attempts

File: src/lbr_fri_ros2_stack/lbr_description/urdf/dual_iiwa7/dual_iiwa7_mod.urdf (robot description, URDF)
Before this commit: robot dual_iiwa7, 19 links, 18 joints
Joints:
- joint world_kuka_green_joint: origin xyz=0.75 0.9 0 rpy=0 0 0 -> xyz=0.75 0.65 0 rpy=0 0 0

Commit message: modified urdf

File: src/lbr_fri_ros2_stack/lbr_description/urdf/dual_iiwa7/dual_iiwa7_mod.urdf (robot description, URDF)
Before this commit: robot dual_iiwa7, 19 links, 18 joints
Joints:
- joint world_kuka_green_joint: origin xyz=0.75 0.65 0 rpy=0 0 0 -> xyz=0.75 0.9 0 rpy=0 0 0

File: src/lbr_fri_ros2_stack/lbr_description/urdf/dual_iiwa7/dual_iiwa7_mod_chisel_gripper.urdf (robot description, URDF)
Before this commit: robot dual_iiwa7, 30 links, 29 joints
Joints:
- joint world_kuka_green_joint: origin xyz=0.75 0.9 0 rpy=0 0 0 -> xyz=0.75 1.1 0 rpy=0 0 0
