Commit message: Added End Effectors

File: src/lbr_fri_ros2_stack/lbr_description/urdf/dual_iiwa7/dual_iiwa7_mod_chisel_gripper.urdf (robot description, URDF)
Before this commit: robot dual_iiwa7, 21 links, 20 joints
Links:
- removed link kuka_blue_link_tcp
- removed link kuka_green_link_tcp
- added link kuka_blue_tcp_link
- added link kuka_green_tcp_link
- added link robotiq_85_base_link, mass 6.6320197e-01; collision mesh filename=file:///home/battery/multi_iiwa_ws/install/robotiq_descript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; visual mesh filename=file:///home/battery/multi_iiwa_ws/install/robotiq_descript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
- added link robotiq_85_left_finger_link, mass 4.260376752e-02; collision mesh filename=file:///home/battery/multi_iiwa_ws/install/robotiq_descript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; visual mesh filename=file:///home/battery/multi_iiwa_ws/install/robotiq_descript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
- added link robotiq_85_left_finger_tip_link, mass 4.268588744e-02; collision mesh filename=file:///home/battery/multi_iiwa_ws/install/robotiq_descript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; visual mesh filename=file:///home/battery/multi_iiwa_ws/install/robotiq_descript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
- added link robotiq_85_left_inner_knuckle_link, mass 2.969376448e-02; collision mesh filename=file:///home/battery/multi_iiwa_ws/install/robotiq_descript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; visual mesh filename=file:///home/battery/multi_iiwa_ws/install/robotiq_descript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
- added link robotiq_85_left_knuckle_link, mass 1.384773208e-02; collision mesh filename=file:///home/battery/multi_iiwa_ws/install/robotiq_descript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; visual mesh filename=file:///home/battery/multi_iiwa_ws/install/robotiq_descript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
- added link robotiq_85_right_finger_link, mass 4.260376752000000e-02; collision mesh filename=file:///home/battery/multi_iiwa_ws/install/robotiq_descript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; visual mesh filename=file:///home/battery/multi_iiwa_ws/install/robotiq_descript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
- added link robotiq_85_right_finger_tip_link, mass 4.268588744e-02; collision mesh filename=file:///home/battery/multi_iiwa_ws/install/robotiq_descript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; visual mesh filename=file:///home/battery/multi_iiwa_ws/install/robotiq_descript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
- added link robotiq_85_right_inner_knuckle_link, mass 2.969376448e-02; collision mesh filename=file:///home/battery/multi_iiwa_ws/install/robotiq_descript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; visual mesh filename=file:///home/battery/multi_iiwa_ws/install/robotiq_descript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
- added link robotiq_85_right_knuckle_link, mass 1.384773208e-02; collision mesh filename=file:///home/battery/multi_iiwa_ws/install/robotiq_descript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; visual mesh filename=file:///home/battery/multi_iiwa_ws/install/robotiq_descript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
- link kuka_blue_link_ee: mass 1.3 -> None; geometry 
- link kuka_green_link_ee: geometry collision mesh filename=package://lbr_description/meshes/iiwa7/collision/chisel.stl scale=0.01 0.01 0.01; visual mesh filename=package://lbr_description/meshes/iiwa7/visual/chisel.dae scale=0.01 0.01 0.01
Joints:
- removed joint kuka_blue_joint_tcp
- removed joint kuka_green_joint_tcp
- added joint kuka_blue_tcp_joint: type fixed, parent kuka_blue_link_ee, child kuka_blue_tcp_link, origin xyz=0 0 0.15 rpy=0 0 0
- added joint kuka_green_tcp_joint: type fixed, parent kuka_green_link_ee, child kuka_green_tcp_link, origin xyz=0 0 0.23 rpy=0 0 0
- added joint robotiq_85_base_joint: type fixed, parent kuka_blue_link_ee, child robotiq_85_base_link, origin xyz=0 0 0 rpy=0 0 0
- added joint robotiq_85_left_finger_joint: type fixed, parent robotiq_85_left_knuckle_link, child robotiq_85_left_finger_link, origin xyz=0.03152616 0.0 -0.00376347 rpy=0 0 0
- added joint robotiq_85_left_finger_tip_joint: type continuous, parent robotiq_85_left_finger_link, child robotiq_85_left_finger_tip_link, origin xyz=0.00563134 0.0 0.04718515 rpy=0 0 0, axis 0 -1 0, mimic joint=robotiq_85_left_knuckle_joint multiplier=-1
- added joint robotiq_85_left_inner_knuckle_joint: type continuous, parent robotiq_85_base_link, child robotiq_85_left_inner_knuckle_link, origin xyz=0.0127 0.0 0.06142 rpy=0 0 0, axis 0 -1 0, mimic joint=robotiq_85_left_knuckle_joint
- added joint robotiq_85_left_knuckle_joint: type revolute, parent robotiq_85_base_link, child robotiq_85_left_knuckle_link, origin xyz=0.03060114 0.0 0.05490452 rpy=0 0 0, axis 0 -1 0, limit lower=0.0 upper=0.8 effort=50 velocity=0.5
- added joint robotiq_85_right_finger_joint: type fixed, parent robotiq_85_right_knuckle_link, child robotiq_85_right_finger_link, origin xyz=-0.03152616 0.0 -0.00376347 rpy=0 0 0
- added joint robotiq_85_right_finger_tip_joint: type continuous, parent robotiq_85_right_finger_link, child robotiq_85_right_finger_tip_link, origin xyz=-0.00563134 0.0 0.04718515 rpy=0 0 0, axis 0 -1 0, mimic joint=robotiq_85_left_knuckle_joint
- added joint robotiq_85_right_inner_knuckle_joint: type continuous, parent robotiq_85_base_link, child robotiq_85_right_inner_knuckle_link, origin xyz=-0.0127 0.0 0.06142 rpy=0 0 0, axis 0 -1 0, mimic joint=robotiq_85_left_knuckle_joint multiplier=-1
- added joint robotiq_85_right_knuckle_joint: type revolute, parent robotiq_85_base_link, child robotiq_85_right_knuckle_link, origin xyz=-0.03060114 0.0 0.05490452 rpy=0 0 0, axis 0 -1 0, limit lower=-0.8 upper=0.0 effort=50 velocity=0.5, mimic joint=robotiq_85_left_knuckle_joint multiplier=-1
- joint world_kuka_blue_joint: origin xyz=0 0 0 rpy=0 0 0 -> xyz=0.7 -0.3 0 rpy=0 0 0
- joint world_kuka_green_joint: origin xyz=1 1 0 rpy=0 0 0 -> xyz=0.75 0.9 0 rpy=0 0 0

Commit message: ..

File: src/lbr_fri_ros2_stack/lbr_description/urdf/dual_iiwa7/dual_iiwa7_mod_chisel_gripper.urdf (robot description, URDF)
Before this commit: robot dual_iiwa7, 30 links, 29 joints
Links:
- removed link kuka_blue_tcp_link
- removed link kuka_green_tcp_link
- added link kuka_blue_link_tcp
- added link kuka_green_link_tcp
Joints:
- removed joint kuka_blue_tcp_joint
- removed joint kuka_green_tcp_joint
- added joint kuka_blue_joint_tcp: type fixed, parent kuka_blue_link_ee, child kuka_blue_link_tcp, origin xyz=0 0 0.15 rpy=0 0 0
- added joint kuka_green_joint_tcp: type fixed, parent kuka_green_link_ee, child kuka_green_link_tcp, origin xyz=0 0 0.23 rpy=0 0 0

Commit message: Added Gripper Mesh files

File: src/lbr_fri_ros2_stack/lbr_description/urdf/dual_iiwa7/dual_iiwa7_mod_chisel_gripper.urdf (robot description, URDF)
Before this commit: robot dual_iiwa7, 30 links, 29 joints
Links:
- link robotiq_85_base_link: geometry collision mesh filename=package://robotiq_description/meshes/collision/2f_85/roboti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; visual mesh filename=package://robotiq_description/meshes/visual/2f_85/robotiq_b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
- link robotiq_85_left_finger_link: geometry collision mesh filename=package://robotiq_description/meshes/collision/2f_85/left_f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; visual mesh filename=package://robotiq_description/meshes/visual/2f_85/left_fing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
- link robotiq_85_left_finger_tip_link: geometry collision mesh filename=package://robotiq_description/meshes/collision/2f_85/left_f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; visual mesh filename=package://robotiq_description/meshes/visual/2f_85/left_fing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
- link robotiq_85_left_inner_knuckle_link: geometry collision mesh filename=package://robotiq_description/meshes/collision/2f_85/left_i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; visual mesh filename=package://robotiq_description/meshes/visual/2f_85/left_inne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
- link robotiq_85_left_knuckle_link: geometry collision mesh filename=package://robotiq_description/meshes/collision/2f_85/left_k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; visual mesh filename=package://robotiq_description/meshes/visual/2f_85/left_knuc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
- link robotiq_85_right_finger_link: geometry collision mesh filename=package://robotiq_description/meshes/collision/2f_85/right_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; visual mesh filename=package://robotiq_description/meshes/visual/2f_85/right_fin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
- link robotiq_85_right_finger_tip_link: geometry collision mesh filename=package://robotiq_description/meshes/collision/2f_85/right_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; visual mesh filename=package://robotiq_description/meshes/visual/2f_85/right_fin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
- link robotiq_85_right_inner_knuckle_link: geometry collision mesh filename=package://robotiq_description/meshes/collision/2f_85/right_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; visual mesh filename=package://robotiq_description/meshes/visual/2f_85/right_inn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
- link robotiq_85_right_knuckle_link: geometry collision mesh filename=package://robotiq_description/meshes/collision/2f_85/right_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; visual mesh filename=package://robotiq_description/meshes/visual/2f_85/right_knu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

Commit message: created new mc package

File: src/lbr_fri_ros2_stack/lbr_description/urdf/dual_iiwa7/dual_iiwa7_mod_chisel_gripper.urdf (robot description, URDF)
Before this commit: robot dual_iiwa7, 30 links, 29 joints
Joints:
- joint robotiq_85_base_joint: origin xyz=0 0 0 rpy=0 0 0 -> xyz=0 0 0 rpy=0 0 1.57

Commit message: added tool calibration for chisel

File: src/lbr_fri_ros2_stack/lbr_description/urdf/dual_iiwa7/dual_iiwa7_mod_chisel_gripper.urdf (robot description, URDF)
Before this commit: robot dual_iiwa7, 30 links, 29 joints
Links:
- link kuka_green_link_ee: mass 0.1 -> 0.55
Joints:
- joint kuka_green_joint_tcp: origin xyz=0 0 0.23 rpy=0 0 0 -> xyz=0.00051 -0.00012 0.23332 rpy=0 0 0

Commit message: ...

File: src/lbr_fri_ros2_stack/lbr_description/urdf/dual_iiwa7/dual_iiwa7_mod_chisel_gripper.urdf (robot description, URDF)
Before this commit: robot dual_iiwa7, 30 links, 29 joints
Joints:
- joint kuka_green_joint_ee: origin xyz=0 0 0.035 rpy=0 0 0 -> xyz=0 0 0.035 rpy=0 0 3.14
- joint world_kuka_green_joint: origin xyz=0.75 1.1 0 rpy=0 0 0 -> xyz=0.8 0.9 -0.15 rpy=0 0 3.14

Commit message: ..

File: src/lbr_fri_ros2_stack/lbr_description/urdf/dual_iiwa7/dual_iiwa7_mod_chisel_gripper.urdf (robot description, URDF)
Before this commit: robot dual_iiwa7, 30 links, 29 joints
Links:
- link kuka_green_link_ee: geometry collision mesh filename=package://lbr_description/meshes/iiwa7/collision/chisel.stl scale=0.001 0.001 0.001; visual mesh filename=package://lbr_description/meshes/iiwa7/visual/chisel.dae scale=0.01 0.01 0.01
Joints:
- joint world_kuka_green_joint: origin xyz=0.8 0.9 -0.15 rpy=0 0 3.14 -> xyz=0.75 0.8 -0.3 rpy=0 0 3.14

Commit message: ..

File: src/lbr_fri_ros2_stack/lbr_description/urdf/dual_iiwa7/dual_iiwa7_mod_chisel_gripper.urdf (robot description, URDF)
Before this commit: robot dual_iiwa7, 30 links, 29 joints
Joints:
- joint world_kuka_green_joint: origin xyz=0.75 0.8 -0.3 rpy=0 0 3.14 -> xyz=0.8 0.7 -0.4 rpy=0 0 -2.356

Commit message: ..

File: src/lbr_fri_ros2_stack/lbr_description/urdf/dual_iiwa7/dual_iiwa7_mod_chisel_gripper.urdf (robot description, URDF)
Before this commit: robot dual_iiwa7, 30 links, 29 joints
Joints:
- joint world_kuka_blue_joint: origin xyz=0.7 -0.3 0 rpy=0 0 0 -> xyz=0.55 -0.35 -0.25 rpy=0 0 0.783

Commit message: ..

File: src/lbr_fri_ros2_stack/lbr_description/urdf/dual_iiwa7/dual_iiwa7_mod_chisel_gripper.urdf (robot description, URDF)
Before this commit: robot dual_iiwa7, 30 links, 29 joints
Joints:
- joint world_kuka_blue_joint: origin xyz=0.55 -0.35 -0.25 rpy=0 0 0.783 -> xyz=0.55 -0.4 -0.25 rpy=0 0 0.783

Commit message: changed urdf to add HIGH positions in kuka xacros

File: src/lbr_fri_ros2_stack/lbr_description/urdf/dual_iiwa7/dual_iiwa7_mod_chisel_gripper.urdf (robot description, URDF)
Before this commit: robot dual_iiwa7, 30 links, 29 joints
Joints:
- joint world_kuka_green_joint: origin xyz=0.8 0.7 -0.4 rpy=0 0 -2.356 -> xyz=0.8 0.7 -0.55 rpy=0 0 -2.356

File: src/lbr_fri_ros2_stack/lbr_description/urdf/kuka_blue/kuka_blue.xacro (robot description, xacro)
@@ -17,5 +17,6 @@
         <parent link="world" />
         <child link="link_0" />
-        <origin xyz="0.55 -0.4 -0.25" rpy="0 0 0.783"/>
+        <!-- <origin xyz="0.55 -0.4 -0.25" rpy="0 0 0.783"/> -->
+        <origin xyz="0.55 -0.4 -0.35" rpy="0 0 0.783"/>
     </joint>
     <!-- iiwa -->

File: src/lbr_fri_ros2_stack/lbr_description/urdf/kuka_green/kuka_green.xacro (robot description, xacro)
@@ -15,5 +15,6 @@
         <parent link="world" />
         <child link="link_0" />
-        <origin xyz="0.8 0.7 -0.4" rpy="0 0 -2.356"/>
+        <!-- <origin xyz="0.8 0.7 -0.4" rpy="0 0 -2.356"/> -->
+        <origin xyz="0.8 0.7 -0.55" rpy="0 0 -2.356"/>
     </joint>
     <!-- iiwa -->
@@ -52,5 +53,5 @@
         <parent link="link_ee"/>
         <child link="link_tcp"/>
-        <origin rpy="0 0 0" xyz="-0.00071 -0.00018 0.11105"/>
+        <origin rpy="0 0 0" xyz="0.00051 -0.00012 0.23332"/>
     </joint>
 </robot>
