Commit message: ..

File: src/lbr_fri_ros2_stack/lbr_description/urdf/iiwa7/iiwa7_description.xacro (robot description, xacro)
@@ -265,5 +265,5 @@
             </collision>
         </link>
-        <joint name="joint_ee" type="fixed">
+        <!-- <joint name="joint_ee" type="fixed">
             <parent link="link_7" />
             <child link="link_ee" />
@@ -271,5 +271,5 @@
         </joint>
         <link name="link_ee">
-        </link>
+        </link> -->
     </xacro:macro>
 </robot>
