Commit message: Used URDF of iiwa_stack for cross-verification

File: src/lbr_fri_ros2_stack/lbr_description/urdf/iiwa7/iiwa7_desc_org_backup.xacro (robot description, xacro)
@@ -24,25 +24,24 @@
         <link name="link_0">
             <inertial>
-                <origin rpy="0 0 0" xyz="-0.1 0 0.07" />
-                <mass value="5" />
-                <inertia ixx="0.05"  ixy="0"  ixz="0" iyy="0.06" iyz="0" izz="0.03"/>
+                <origin rpy="0 0 0" xyz="-0.012857 0.0 0.069964" />
+                <mass value="4.855658" />
+                <inertia ixx="0.017839" ixy="0.0" ixz="0.000781" iyy="0.022294" iyz="0.0"
+                    izz="0.021334" />
             </inertial>
             <visual>
                 <origin rpy="0 0 0" xyz="0 0 0" />
                 <geometry>
-                    <mesh filename="package://iiwa7_description/meshes/iiwa7/visual/link_0.stl" />
-                </geometry>
-                <material name="Grey"/>
+                    <mesh filename="package://lbr_description/meshes/iiwa7/visual/link_0.dae" />
+                </geometry>
             </visual>
             <collision>
                 <origin rpy="0 0 0" xyz="0 0 0" />
                 <geometry>
-                    <mesh filename="package://iiwa7_description/meshes/iiwa7/collision/link_0.stl" />
-                </geometry>
-                <material name="Grey"/>
+                    <mesh filename="package://lbr_description/meshes/iiwa7/collision/link_0.stl" />
+                </geometry>
             </collision>
         </link>
         <joint name="A1" type="revolute">
-            <origin rpy="0 0 0" xyz="0.0 0.0 0.15" />
+            <origin rpy="0 0 0" xyz="0.0 0.0 0.1475" />
             <parent link="link_0" />
             <child link="link_1" />
@@ -57,28 +56,27 @@
         <link name="link_1">
             <inertial>
-                <origin rpy="0 0 0" xyz="0.0 -0.03 0.12" />
-                <mass value="3.4525" />
-                <inertia ixx="0.02183" ixy="0.0" ixz="0.0" iyy="0.007703" iyz="-0.003887" izz="0.02083"/>
-            </inertial>
-            <visual>
-                <origin rpy="0 0 0" xyz="0.0 0.0 0.0075" />
-                <geometry>
-                    <mesh filename="package://iiwa7_description/meshes/iiwa7/visual/link_1.stl" />
-                </geometry>
-                <material name="Orange"/>
-            </visual>
-            <collision>
-                <origin rpy="0 0 0" xyz="0.0 0.0 0.0075" />
-                <geometry>
-                    <mesh filename="package://iiwa7_description/meshes/iiwa7/collision/link_1.stl" />
-                </geometry>
-                <material name="Orange"/>
+                <origin rpy="0 0 0" xyz="0.0 -0.034819 0.123299" />
+                <mass value="3.394011" />
+                <inertia ixx="0.021383" ixy="0.0" ixz="0.0" iyy="0.020403" iyz="0.003797"
+                    izz="0.007563" />
+            </inertial>
+            <visual>
+                <origin rpy="0 0 0" xyz="0.0 0.0 -0.1475" />
+                <geometry>
+                    <mesh filename="package://lbr_description/meshes/iiwa7/visual/link_1.dae" />
+                </geometry>
+            </visual>
+            <collision>
+                <origin rpy="0 0 0" xyz="0.0 0.0 -0.1475" />
+                <geometry>
+                    <mesh filename="package://lbr_description/meshes/iiwa7/collision/link_1.stl" />
+                </geometry>
             </collision>
         </link>
         <joint name="A2" type="revolute">
-            <origin rpy="${PI / 2}   0 ${PI}" xyz="0.0 0.0 0.19" />
+            <origin rpy="0 0 0" xyz="0.0 -0.0105 0.1925" />
             <parent link="link_1" />
             <child link="link_2" />
-            <axis xyz="0.0 0.0 1.0" />
+            <axis xyz="0.0 1.0 0.0" />
             <limit
                 effort="${joint_limits['A2']['effort']}"
@@ -90,25 +88,24 @@
         <link name="link_2">
             <inertial>
-                <origin rpy="0 0 0" xyz="0.0003 0.059 0.042" />
-                <mass value="3.4821" />
-                <inertia ixx="0.02076"  ixy="0"  ixz="-0.003626" iyy="0.02179" iyz="0" izz="0.00779"/>
-            </inertial>
-            <visual>
-                <origin rpy="0 0 0" xyz="0.0 0.0 0.0" />
-                <geometry>
-                    <mesh filename="package://iiwa7_description/meshes/iiwa7/visual/link_2.stl" />
-                </geometry>
-                <material name="Orange"/>
-            </visual>
-            <collision>
-                <origin rpy="0 0 0" xyz="0.0 0.0 0.0" />
-                <geometry>
-                    <mesh filename="package://iiwa7_description/meshes/iiwa7/collision/link_2.stl" />
-                </geometry>
-                <material name="Orange"/>
+                <origin rpy="0 0 0" xyz="0.0 0.039793 0.086944" />
+                <mass value="4.031991" />
+                <inertia ixx="0.031697" ixy="0.0" ixz="0.0" iyy="0.03008" iyz="0.005889"
+                    izz="0.009666" />
+            </inertial>
+            <visual>
+                <origin rpy="0 0 0" xyz="0.0 0.0105 -0.34" />
+                <geometry>
+                    <mesh filename="package://lbr_description/meshes/iiwa7/visual/link_2.dae" />
+                </geometry>
+            </visual>
+            <collision>
+                <origin rpy="0 0 0" xyz="0.0 0.0105 -0.34" />
+                <geometry>
+                    <mesh filename="package://lbr_description/meshes/iiwa7/collision/link_2.stl" />
+                </geometry>
             </collision>
         </link>
         <joint name="A3" type="revolute">
-            <origin rpy="${PI / 2} 0 ${PI}" xyz="0.0 0.21 0.0" />
+            <origin rpy="0 0 0" xyz="0.0 0.0105 0.2075" />
             <parent link="link_2" />
             <child link="link_3" />
@@ -123,28 +120,27 @@
         <link name="link_3">
             <inertial>
-                <origin rpy="0 0 0" xyz="0 0.03 0.13" />
-                <mass value="4.05623" />
-                <inertia ixx="0.03204"  ixy="0"  ixz="0" iyy="0.00972" iyz="0.006227" izz="0.03042"/>
-            </inertial>
-            <visual>
-                <origin rpy="0 0 0" xyz="0.0 0.0 -0.026" />
-                <geometry>
-                    <mesh filename="package://iiwa7_description/meshes/iiwa7/visual/link_3.stl" />
-                </geometry>
-                <material name="Orange"/>
-            </visual>
-            <collision>
-                <origin rpy="0 0 0" xyz="0.0 0.0 -0.026" />
-                <geometry>
-                    <mesh filename="package://iiwa7_description/meshes/iiwa7/collision/link_3.stl" />
-                </geometry>
-                <material name="Orange"/>
+                <origin rpy="0 0 0" xyz="0.0 0.034819 0.123299" />
+                <mass value="3.394011" />
+                <inertia ixx="0.021383" ixy="0.0" ixz="0.0" iyy="0.020403" iyz="-0.003797"
+                    izz="0.007563" />
+            </inertial>
+            <visual>
+                <origin rpy="0 0 0" xyz="0.0 0.0 -0.5475" />
+                <geometry>
+                    <mesh filename="package://lbr_description/meshes/iiwa7/visual/link_3.dae" />
+                </geometry>
+            </visual>
+            <collision>
+                <origin rpy="0 0 0" xyz="0.0 0.0 -0.5475" />
+                <geometry>
+                    <mesh filename="package://lbr_description/meshes/iiwa7/collision/link_3.stl" />
+                </geometry>
             </collision>
         </link>
         <joint name="A4" type="revolute">
-            <origin rpy="${PI / 2} 0 0" xyz="0.0 0.0 0.19" />
+            <origin rpy="0 0 0" xyz="0.0 0.0105 0.1925" />
             <parent link="link_3" />
             <child link="link_4" />
-            <axis xyz="0.0 0.0 1.0" />
+            <axis xyz="0.0 -1.0 0.0" />
             <limit
                 effort="${joint_limits['A4']['effort']}"
@@ -156,25 +152,24 @@
         <link name="link_4">
             <inertial>
-                <origin rpy="0 0 0" xyz="0 0.067 0.034" />
-                <mass value="3.4822" />
-                <inertia ixx="0.02178"  ixy="0"  ixz="0" iyy="0.02075" iyz="-0.003625" izz="0.007785" />
-            </inertial>
-            <visual>
-                <origin rpy="0 0 0" xyz="0 0 0" />
-                <geometry>
-                    <mesh filename="package://iiwa7_description/meshes/iiwa7/visual/link_4.stl" />
-                </geometry>
-                <material name="Orange"/>
-            </visual>
-            <collision>
-                <origin rpy="0 0 0" xyz="0 0 0" />
-                <geometry>
-                    <mesh filename="package://iiwa7_description/meshes/iiwa7/collision/link_4.stl" />
-                </geometry>
-                <material name="Orange"/>
+                <origin rpy="0 0 0" xyz="0.0 -0.039793 0.086944" />
+                <mass value="4.031989" />
+                <inertia ixx="0.031695" ixy="0.0" ixz="0.0" iyy="0.030079" iyz="-0.005889"
+                    izz="0.009665" />
+            </inertial>
+            <visual>
+                <origin rpy="0 0 0" xyz="0.0 -0.0105 -0.74" />
+                <geometry>
+                    <mesh filename="package://lbr_description/meshes/iiwa7/visual/link_4.dae" />
+                </geometry>
+            </visual>
+            <collision>
+                <origin rpy="0 0 0" xyz="0.0 -0.0105 -0.74" />
+                <geometry>
+                    <mesh filename="package://lbr_description/meshes/iiwa7/collision/link_4.stl" />
+                </geometry>
             </collision>
         </link>
         <joint name="A5" type="revolute">
-            <origin rpy="${-PI / 2} ${PI} 0" xyz="0.0 0.21 0.0" />
+            <origin rpy="0 0 0" xyz="0.0 -0.0105 0.2075" />
             <parent link="link_4" />
             <child link="link_5" />
@@ -189,28 +184,27 @@
         <link name="link_5">
             <inertial>
-                <origin rpy="0 0 0" xyz="0.0001 0.021 0.076" />
-                <mass value="2.1633" />
-                <inertia ixx="0.01287"  ixy="0"  ixz="0" iyy="0.005708" iyz="-0.003946" izz="0.01112" />
-            </inertial>
-            <visual>
-                <origin rpy="0 0 0" xyz="0 0 -0.026" />
-                <geometry>
-                    <mesh filename="package://iiwa7_description/meshes/iiwa7/visual/link_5.stl" />
-                </geometry>
-                <material name="Orange"/>
-            </visual>
-            <collision>
-                <origin rpy="0 0 0" xyz="0 0 -0.026" />
-                <geometry>
-                    <mesh filename="package://iiwa7_description/meshes/iiwa7/collision/link_5.stl" />
-                </geometry>
-                <material name="Orange"/>
+                <origin rpy="0 0 0" xyz="0.0 -0.029824 0.076267" />
+                <mass value="1.529239" />
+                <inertia ixx="0.008485" ixy="0.0" ixz="0.0" iyy="0.007136" iyz="0.002806"
+                    izz="0.003848" />
+            </inertial>
+            <visual>
+                <origin rpy="0 0 0" xyz="0.0 0.0 -0.9475" />
+                <geometry>
+                    <mesh filename="package://lbr_description/meshes/iiwa7/visual/link_5.dae" />
+                </geometry>
+            </visual>
+            <collision>
+                <origin rpy="0 0 0" xyz="0.0 0.0 -0.9475" />
+                <geometry>
+                    <mesh filename="package://lbr_description/meshes/iiwa7/collision/link_5.stl" />
+                </geometry>
             </collision>
         </link>
         <joint name="A6" type="revolute">
-            <origin rpy="${PI / 2} 0 0" xyz="0 0.06070 0.19" />
+            <origin rpy="0 0 0" xyz="0.0 -0.0707 0.1925" />
             <parent link="link_5" />
             <child link="link_6" />
-            <axis xyz="0.0 0.0 1.0" />
+            <axis xyz="0.0 1.0 0.0" />
             <limit
                 effort="${joint_limits['A6']['effort']}"
@@ -222,25 +216,24 @@
         <link name="link_6">
             <inertial>
-                <origin rpy="0 0 0" xyz="0 0.0006 0.0004" />
-                <mass value="2.3466" />
-                <inertia ixx="0.006509"  ixy="0"  ixz="0" iyy="0.006259" iyz="0.00031891" izz="0.004527" />
-            </inertial>
-            <visual>
-                <origin rpy="0 0 0" xyz="0 0 0" />
-                <geometry>
-                    <mesh filename="package://iiwa7_description/meshes/iiwa7/visual/link_6.stl" />
-                </geometry>
-                <material name="Orange"/>
-            </visual>
-            <collision>
-                <origin rpy="0 0 0" xyz="0 0 0" />
-                <geometry>
-                    <mesh filename="package://iiwa7_description/meshes/iiwa7/collision/link_6.stl" />
-                </geometry>
-                <material name="Orange"/>
+                <origin rpy="0 0 0" xyz="0.0 0.07102 0.00495" />
+                <mass value="2.403626" />
+                <inertia ixx="0.007067" ixy="0.0" ixz="0.0" iyy="0.006804" iyz="0.000311"
+                    izz="0.004629" />
+            </inertial>
+            <visual>
+                <origin rpy="0 0 0" xyz="0.0 0.0707 -1.14" />
+                <geometry>
+                    <mesh filename="package://lbr_description/meshes/iiwa7/visual/link_6.dae" />
+                </geometry>
+            </visual>
+            <collision>
+                <origin rpy="0 0 0" xyz="0.0 0.0707 -1.14" />
+                <geometry>
+                    <mesh filename="package://lbr_description/meshes/iiwa7/collision/link_6.stl" />
+                </geometry>
             </collision>
         </link>
         <joint name="A7" type="revolute">
-            <origin rpy="${- PI / 2} ${PI} 0" xyz="0 0.081 0.06070" />
+            <origin rpy="0 0 0" xyz="0.0 0.0707 0.091" />
             <parent link="link_6" />
             <child link="link_7" />
@@ -255,21 +248,19 @@
         <link name="link_7">
             <inertial>
-                <origin rpy="0 0 0" xyz="0 0 0.02" />
-                <mass value="3.129" />
-                <inertia ixx="0.01464"  ixy="0.0005912"  ixz="0" iyy="0.01465" iyz="0" izz="0.002872" />
-            </inertial>
-            <visual>
-                <origin rpy="0 0 0" xyz="0 0 -0.0005" />
-                <geometry>
-                    <mesh filename="package://iiwa7_description/meshes/iiwa7/visual/link_7.stl" />
-                </geometry>
-                <material name="Grey"/>
-            </visual>
-            <collision>
-                <origin rpy="0 0 0" xyz="0 0 -0.0005" />
-                <geometry>
-                    <mesh filename="package://iiwa7_description/meshes/iiwa7/collision/link_7.stl" />
-                </geometry>
-                <material name="Grey"/>
+                <origin rpy="0 0 0" xyz="3.0000e-06 -2.0000e-06 1.3782e-02" />
+                <mass value="0.259474" />
+                <inertia ixx="0.000171" ixy="0.0" ixz="0.0" iyy="0.000171" iyz="0.0" izz="0.000299" />
+            </inertial>
+            <visual>
+                <origin rpy="0 0 0" xyz="0.0 0.0 -1.231" />
+                <geometry>
+                    <mesh filename="package://lbr_description/meshes/iiwa7/visual/link_7.dae" />
+                </geometry>
+            </visual>
+            <collision>
+                <origin rpy="0 0 0" xyz="0.0 0.0 -1.231" />
+                <geometry>
+                    <mesh filename="package://lbr_description/meshes/iiwa7/collision/link_7.stl" />
+                </geometry>
             </collision>
         </link>

File: src/lbr_fri_ros2_stack/lbr_description/urdf/kuka_blue/_backup.xacro (robot description, xacro)
@@ -3,8 +3,9 @@
 <robot name="iiwa7" xmlns:xacro="http://www.ros.org/wiki/xacro">
     <!-- include the lbr iiwa macro -->
-    <xacro:include filename="$(find lbr_description)/urdf/iiwa7/materials.xacro" />
     <xacro:include filename="$(find lbr_description)/urdf/iiwa7/iiwa7_description.xacro" />
+    <xacro:include filename="$(find robotiq_description)/urdf/robotiq_2f_85_macro.urdf.xacro" />
     <xacro:arg name="robot_name" default="lbr" />
     <xacro:arg name="sim" default="true" />
+    <xacro:arg name="use_fake_hardware" default="true" />
     <xacro:arg
         name="system_parameters_path"
@@ -16,10 +17,8 @@
         <parent link="world" />
         <child link="link_0" />
-        <!-- <origin xyz="0.8 0.7 -0.4" rpy="0 0 -2.356"/> -->
-        <!-- <origin xyz="0.8 0.7 -0.55" rpy="0 0 -2.356"/> -->
-        <!-- <origin xyz="0.8 0.7 -0.425" rpy="0 0 -2.356"/> -->
-        <!-- <origin xyz="0.8 0.7 -0.47" rpy="0 0 -2.356"/> -->
-        <!-- <origin xyz="0.85 0.60 -0.46" rpy="0 0 -2.356"/> -->
-        <origin xyz="0 0 0" rpy="0 0 0"/>
+        <!-- <origin xyz="0.55 -0.4 -0.25" rpy="0 0 0.783"/> -->
+        <!-- <origin xyz="0.55 -0.4 -0.35" rpy="0 0 0.783"/> -->
+        <origin xyz="0.55 -0.4 -0.264" rpy="0 0 0.783"/>
+        <!-- <origin xyz="0.6 -0.5 -0.299" rpy="0 0 0.783"/> -->
     </joint>
     <!-- iiwa -->
@@ -30,36 +29,32 @@
     <!-- End Effector -->
     <link name="link_ee">
-        <inertial>
-            <origin rpy="1.57 0 1.57" xyz="0 0 0.055525" />
+        <!-- <inertial>
+            <origin rpy="1.57 0 1.57" xyz="0 0 0.08524" />
             <mass value="0.55" />
             <inertia ixx="0.0001" ixy="0.0" ixz="0.0" iyy="0.0001" iyz="0.0" izz="0.0001" />
         </inertial>
         <visual>
-            <origin rpy="1.57 0 1.57" xyz="0.0 0.0 0.0" />
+            <origin rpy="1.57 0 1.57" xyz="-0.0925 0 0.035" />
             <geometry>
-                <mesh filename="package://lbr_description/meshes/iiwa7/visual/chisel.dae" scale="0.01 0.01 0.01"/>
+                <mesh filename="package://lbr_description/meshes/iiwa7/collision/robotiq_gripper.stl" scale="0.001 0.001 0.001"/>
             </geometry>
-            <material name="Black"/>
         </visual>
         <collision>
-            <origin rpy="1.57 0 1.57" xyz="0.0 0.0 0.0" />
+            <origin rpy="1.57 0 1.57" xyz="-0.0925 0 0.035" />
             <geometry>
-                <mesh filename="package://lbr_description/meshes/iiwa7/collision/chisel.stl" scale="0.001 0.001 0.001"/>
+                <mesh filename="package://lbr_description/meshes/iiwa7/collision/robotiq_gripper.stl" scale="0.001 0.001 0.001"/>
             </geometry>
-            <material name="Black"/>
-        </collision>
+        </collision> -->
     </link>
     <joint name="joint_ee" type="fixed">
         <parent link="link_7"/>
         <child link="link_ee"/>
-        <origin rpy="0 0 3.14" xyz="0 0 0.045"/>
+        <origin rpy="0 0 0" xyz="0 0 0"/>
     </joint>
-    <!-- TCP Link -->
-    <link name="link_tcp"/>
+    <!-- <link name="link_tcp"/>
     <joint name="joint_tcp" type="fixed">
         <parent link="link_ee"/>
         <child link="link_tcp"/>
-        <!-- <origin rpy="0 0 0" xyz="0.00051 -0.00012 0.23332"/> -->
-        <origin rpy="0 0 0" xyz="0.00051 -0.00012 0.23332"/>
-    </joint>
+        <origin rpy="0 0 0" xyz="-0.00022 0.00163 0.17048"/>
+    </joint> -->
 </robot>

File: src/lbr_fri_ros2_stack/lbr_description/urdf/kuka_blue/kuka_blue.xacro (robot description, xacro)
@@ -3,4 +3,5 @@
 <robot name="iiwa7" xmlns:xacro="http://www.ros.org/wiki/xacro">
     <!-- include the lbr iiwa macro -->
+    <xacro:include filename="$(find iiwa7_description)/urdf/materials.xacro" />
     <xacro:include filename="$(find lbr_description)/urdf/iiwa7/iiwa7_description.xacro" />
     <xacro:include filename="$(find robotiq_description)/urdf/robotiq_2f_85_macro.urdf.xacro" />
@@ -35,14 +36,16 @@
         </inertial>
         <visual>
-            <origin rpy="1.57 0 1.57" xyz="-0.0925 0 0.035" />
+            <origin rpy="1.57 0 1.57" xyz="-0.0925 0 0.045" />
             <geometry>
                 <mesh filename="package://lbr_description/meshes/iiwa7/collision/robotiq_gripper.stl" scale="0.001 0.001 0.001"/>
             </geometry>
+            <material name="Black"/>
         </visual>
         <collision>
-            <origin rpy="1.57 0 1.57" xyz="-0.0925 0 0.035" />
+            <origin rpy="1.57 0 1.57" xyz="-0.0925 0 0.045" />
             <geometry>
                 <mesh filename="package://lbr_description/meshes/iiwa7/collision/robotiq_gripper.stl" scale="0.001 0.001 0.001"/>
             </geometry>
+            <material name="Black"/>
         </collision>
     </link>

File: src/lbr_fri_ros2_stack/lbr_description/urdf/kuka_green/kuka_green_mod.xacro (robot description, xacro)
@@ -3,5 +3,4 @@
 <robot name="iiwa7" xmlns:xacro="http://www.ros.org/wiki/xacro">
     <!-- include the lbr iiwa macro -->
-    <xacro:include filename="$(find lbr_description)/urdf/iiwa7/materials.xacro" />
     <xacro:include filename="$(find lbr_description)/urdf/iiwa7/iiwa7_description.xacro" />
     <xacro:arg name="robot_name" default="lbr" />
@@ -20,6 +19,5 @@
         <!-- <origin xyz="0.8 0.7 -0.425" rpy="0 0 -2.356"/> -->
         <!-- <origin xyz="0.8 0.7 -0.47" rpy="0 0 -2.356"/> -->
-        <!-- <origin xyz="0.85 0.60 -0.46" rpy="0 0 -2.356"/> -->
-        <origin xyz="0 0 0" rpy="0 0 0"/>
+        <origin xyz="0.85 0.60 -0.46" rpy="0 0 -2.356"/>
     </joint>
     <!-- iiwa -->
@@ -40,5 +38,4 @@
                 <mesh filename="package://lbr_description/meshes/iiwa7/visual/chisel.dae" scale="0.01 0.01 0.01"/>
             </geometry>
-            <material name="Black"/>
         </visual>
         <collision>
@@ -47,5 +44,4 @@
                 <mesh filename="package://lbr_description/meshes/iiwa7/collision/chisel.stl" scale="0.001 0.001 0.001"/>
             </geometry>
-            <material name="Black"/>
         </collision>
     </link>
@@ -53,5 +49,5 @@
         <parent link="link_7"/>
         <child link="link_ee"/>
-        <origin rpy="0 0 3.14" xyz="0 0 0.045"/>
+        <origin rpy="0 0 3.14" xyz="0 0 0.035"/>
     </joint>
     <!-- TCP Link -->
