Commit message: Improve multi-robot support and URDF namespacing
Refactor URDF descriptions and control configurations to support multiple robot instances by introducing proper namespacing for joints and links.

Updates include:
- Enables robot-specific port IDs in the hardware interface.
- Dynamically defines chain roots and tips based on the robot name for force-torque sensors.
- Standardizes link and joint naming conventions using the robot prefix to prevent collisions in multi-robot setups.
- Improves the base joint definition to ensure correct integration with the world frame.

File: src/lbr_fri_ros2_stack/lbr_description/urdf/iiwa7/iiwa7_description_mod.xacro (robot description, xacro)
@@ -10,16 +10,16 @@
         <xacro:property name="joint_limits_path"
             value="$(find lbr_description)/urdf/iiwa7/joint_limits.yaml" />
-        <xacro:property name="joint_limits" value="${xacro.load_yaml(joint_limits_path)}" />
+        <xacro:property name="base_joint_limits" value="${xacro.load_yaml(joint_limits_path)}" />
         <!-- Keep the YAML generic while exposing prefixed keys to the prefixed model/control macros. -->
         <xacro:property
             name="joint_limits"
             value="${dict([
-                (robot_name + '_' + 'A1', joint_limits['A1']),
-                (robot_name + '_' + 'A2', joint_limits['A2']),
-                (robot_name + '_' + 'A3', joint_limits['A3']),
-                (robot_name + '_' + 'A4', joint_limits['A4']),
-                (robot_name + '_' + 'A5', joint_limits['A5']),
-                (robot_name + '_' + 'A6', joint_limits['A6']),
-                (robot_name + '_' + 'A7', joint_limits['A7']),
+                (robot_name + '_' + 'A1', base_joint_limits['A1']),
+                (robot_name + '_' + 'A2', base_joint_limits['A2']),
+                (robot_name + '_' + 'A3', base_joint_limits['A3']),
+                (robot_name + '_' + 'A4', base_joint_limits['A4']),
+                (robot_name + '_' + 'A5', base_joint_limits['A5']),
+                (robot_name + '_' + 'A6', base_joint_limits['A6']),
+                (robot_name + '_' + 'A7', base_joint_limits['A7']),
             ])}" />
         <!-- constants -->

File: src/lbr_fri_ros2_stack/lbr_description/urdf/kuka_blue/kuka_blue.xacro (robot description, xacro)
@@ -6,23 +6,23 @@
     <!-- <xacro:include filename="$(find robotiq_description)/urdf/robotiq_2f_85_macro.urdf.xacro" /> -->
     <xacro:arg name="sim" default="true" />
-    <xacro:arg name="use_fake_hardware" default="true" />
     <xacro:arg
         name="system_parameters_path"
         default="$(find lbr_ros2_control)/config/lbr_system_parameters.yaml" />
+    <xacro:arg name="robot_name" default="kuka_blue" />
+    <xacro:property name="robot_prefix" value="$(arg robot_name)" />
     <!-- fixed to world, see http://classic.gazebosim.org/tutorials?tut=ros_urdf&cat=connect_ros -->
-    <link name="world">
-        <origin xyz="0 0 0" rpy="0 0 0"/>
-    </link>
-    <xacro:arg name="robot_name" default="kuka_blue" />
+    <link name="world" />
+    <joint name="${robot_prefix}_world_joint" type="fixed">
+        <parent link="world" />
+        <child link="${robot_prefix}_link_0" />
+        <origin xyz="0 0 0" rpy="0 0 0" />
+    </joint>
     <!-- iiwa -->
     <xacro:iiwa7
         robot_name="$(arg robot_name)"
-        parent = "world"
         sim="$(arg sim)"
         system_parameters_path="$(arg system_parameters_path)" />
-        <origin xyz="0 0 0" rpy="0 0 0"/>
-    </xacro:iiwa7>
     <!-- End Effector -->
-    <link name="link_ee">
+    <link name="${robot_prefix}_link_ee">
         <inertial>
             <origin rpy="1.57 0 1.57" xyz="0 0 0.055525" />
@@ -43,14 +43,14 @@
         </collision>
     </link>
-    <joint name="joint_ee" type="fixed">
-        <parent link="link_7"/>
-        <child link="link_ee"/>
+    <joint name="${robot_prefix}_joint_ee" type="fixed">
+        <parent link="${robot_prefix}_link_7"/>
+        <child link="${robot_prefix}_link_ee"/>
         <origin rpy="0 0 3.14" xyz="0 0 0.035"/>
     </joint>
     <!-- TCP Link -->
-    <link name="link_tcp"/>
-    <joint name="joint_tcp" type="fixed">
-        <parent link="link_ee"/>
-        <child link="link_tcp"/>
+    <link name="${robot_prefix}_link_tcp"/>
+    <joint name="${robot_prefix}_joint_tcp" type="fixed">
+        <parent link="${robot_prefix}_link_ee"/>
+        <child link="${robot_prefix}_link_tcp"/>
         <!-- <origin rpy="0 0 0" xyz="0.00051 -0.00012 0.23332"/> NO FORCE TOOL -->
         <!-- <origin rpy="0 0 0" xyz="0.00243 0.0003 0.22498"/> -->

File: src/lbr_fri_ros2_stack/lbr_ros2_control/config/lbr_system_interface_mod.xacro (robot description, xacro)
@@ -17,5 +17,5 @@
                     <plugin>lbr_ros2_control::SystemInterface</plugin>
                     <param name="client_command_mode">${system_parameters['hardware']['client_command_mode']}</param>
-                    <param name="port_id">${system_parameters['hardware']['port_id']}</param>
+                    <param name="port_id">${system_parameters['hardware'].get(robot_name + '_port_id', system_parameters['hardware']['port_id'])}</param>
                     <param name="remote_host">${system_parameters['hardware']['remote_host']}</param>
                     <param name="rt_prio">${system_parameters['hardware']['rt_prio']}</param>
@@ -52,6 +52,6 @@
                 <sensor
                     name="estimated_ft_sensor">
-                    <param name="chain_root">${system_parameters['estimated_ft_sensor']['chain_root']}</param>
-                    <param name="chain_tip">${system_parameters['estimated_ft_sensor']['chain_tip']}</param>
+                    <param name="chain_root">${robot_name + '_link_0'}</param>
+                    <param name="chain_tip">${robot_name + '_link_ee'}</param>
                     <param name="damping">${system_parameters['estimated_ft_sensor']['damping']}</param>
                     <param name="force_x_th">${system_parameters['estimated_ft_sensor']['force_x_th']}</param>
