Commit message: some xacro change to offset world

File: src/lbr_fri_ros2_stack/lbr_description/urdf/kuka_green/kuka_green.xacro (robot description, xacro)
@@ -22,5 +22,6 @@
         <!-- <origin xyz="0 0 0" rpy="0 0 0"/> -->
         <!-- <origin xyz="0.8057409 0.6804944 -0.4295127" rpy="-0.0265684 0.0060622 -2.3834002"/> -->
-        <origin xyz="0.7947345 0.694259 -0.4280015" rpy="-0.0227401 0.0105353 -2.3640002"/>
+        <!-- <origin xyz="0.7947345 0.694259 -0.4280015" rpy="-0.0227401 0.0105353 -2.3640002"/> -->
+        <origin xyz="0.7947345 0.694259 -0.4480015" rpy="-0.0227401 0.0105353 -2.3640002"/>
     </joint>
     <!-- iiwa -->

Commit message: New addons

File: src/lbr_fri_ros2_stack/lbr_description/urdf/kuka_green/kuka_green.xacro (robot description, xacro)
@@ -23,5 +23,6 @@
         <!-- <origin xyz="0.8057409 0.6804944 -0.4295127" rpy="-0.0265684 0.0060622 -2.3834002"/> -->
         <!-- <origin xyz="0.7947345 0.694259 -0.4280015" rpy="-0.0227401 0.0105353 -2.3640002"/> -->
-        <origin xyz="0.7947345 0.694259 -0.4480015" rpy="-0.0227401 0.0105353 -2.3640002"/>
+        <!-- <origin xyz="0.7947345 0.694259 -0.4480015" rpy="-0.0227401 0.0105353 -2.3640002"/>  Friday -->
+        <origin xyz="0.7947345 0.694259 -0.4580015" rpy="-0.0227401 0.0105353 -2.3640002"/>
     </joint>
     <!-- iiwa -->
@@ -60,5 +61,6 @@
         <parent link="link_ee"/>
         <child link="link_tcp"/>
-        <origin rpy="0 0 0" xyz="0.00051 -0.00012 0.23332"/>
+        <!-- <origin rpy="0 0 0" xyz="0.00051 -0.00012 0.23332"/> NO FORCE TOOL -->
+        <origin rpy="0 0 0" xyz="0.00243 0.0003 0.22498"/>
     </joint>
 </robot>

Commit message: Minor Changes

File: src/lbr_fri_ros2_stack/lbr_description/urdf/kuka_green/kuka_green.xacro (robot description, xacro)
@@ -60,5 +60,6 @@
         <parent link="link_ee"/>
         <child link="link_tcp"/>
-        <origin rpy="0 0 0" xyz="0.00051 -0.00012 0.23332"/>
+        <!-- <origin rpy="0 0 0" xyz="0.00051 -0.00012 0.23332"/> NO FORCE CHISEL-->
+        <origin rpy="0 0 0" xyz="0.00243 0.0003 0.22498"/>
     </joint>
 </robot>

Commit message: added code to make ati-sensor-compatible

File: src/lbr_fri_ros2_stack/lbr_description/urdf/kuka_green/kuka_green.xacro (robot description, xacro)
@@ -22,5 +22,5 @@
         <!-- <origin xyz="0 0 0" rpy="0 0 0"/> -->
         <!-- <origin xyz="0.8057409 0.6804944 -0.4295127" rpy="-0.0265684 0.0060622 -2.3834002"/> -->
-        <!-- <origin xyz="0.7947345 0.694259 -0.4280015" rpy="-0.0227401 0.0105353 -2.3640002"/> -->
+        <!-- <origin xyz="0.7947345 0.694259 -0.4280015" rpy="-0.0227401 0.0105353 -2.3640002"/> ORIGINAL-->
         <!-- <origin xyz="0.7947345 0.694259 -0.4480015" rpy="-0.0227401 0.0105353 -2.3640002"/>  Friday -->
         <origin xyz="0.7947345 0.694259 -0.4580015" rpy="-0.0227401 0.0105353 -2.3640002"/>
