Commit message: before demo

File: src/lbr_fri_ros2_stack/lbr_description/urdf/kuka_blue/kuka_blue.xacro (robot description, xacro)
@@ -18,5 +18,7 @@
         <child link="link_0" />
         <!-- <origin xyz="0.55 -0.4 -0.25" rpy="0 0 0.783"/> -->
-        <origin xyz="0.55 -0.4 -0.35" rpy="0 0 0.783"/>
+        <!-- <origin xyz="0.55 -0.4 -0.35" rpy="0 0 0.783"/> -->
+        <origin xyz="0.55 -0.4 -0.264" rpy="0 0 0.783"/>
+        <!-- <origin xyz="0.6 -0.5 -0.299" rpy="0 0 0.783"/> -->
     </joint>
     <!-- iiwa -->

File: src/lbr_fri_ros2_stack/lbr_description/urdf/kuka_green/kuka_green.xacro (robot description, xacro)
@@ -16,5 +16,8 @@
         <child link="link_0" />
         <!-- <origin xyz="0.8 0.7 -0.4" rpy="0 0 -2.356"/> -->
-        <origin xyz="0.8 0.7 -0.55" rpy="0 0 -2.356"/>
+        <!-- <origin xyz="0.8 0.7 -0.55" rpy="0 0 -2.356"/> -->
+        <!-- <origin xyz="0.8 0.7 -0.425" rpy="0 0 -2.356"/> -->
+        <!-- <origin xyz="0.8 0.7 -0.47" rpy="0 0 -2.356"/> -->
+        <origin xyz="0.85 0.60 -0.46" rpy="0 0 -2.356"/>
     </joint>
     <!-- iiwa -->
@@ -53,4 +56,5 @@
         <parent link="link_ee"/>
         <child link="link_tcp"/>
+        <!-- <origin rpy="0 0 0" xyz="0.00051 -0.00012 0.23332"/> -->
         <origin rpy="0 0 0" xyz="0.00051 -0.00012 0.23332"/>
     </joint>

Commit message: calibrated blue and green kuka for motive (using -WIS PC)

File: src/lbr_fri_ros2_stack/lbr_description/urdf/kuka_blue/kuka_blue.xacro (robot description, xacro)
@@ -19,6 +19,13 @@
         <!-- <origin xyz="0.55 -0.4 -0.25" rpy="0 0 0.783"/> -->
         <!-- <origin xyz="0.55 -0.4 -0.35" rpy="0 0 0.783"/> -->
-        <origin xyz="0.55 -0.4 -0.264" rpy="0 0 0.783"/>
-        <!-- <origin xyz="0.6 -0.5 -0.299" rpy="0 0 0.783"/> -->
+        <!-- <origin xyz="0.55 -0.4 -0.264" rpy="0 0 0.783"/>   CORRECT VALUE USED ON FRIDAY DEMO -->
+        <!-- <origin xyz="0.5796 -0.4125 -0.2668" rpy="0.74287 -0.01400 0.029986"/> RS -->
+        <!-- <origin xyz="0.5796 -0.4125 -0.2668" rpy="0.03155910360450854 0.00996866505764844 0.7429270934423268"/>  RS-->
+        <!-- <origin xyz="0.5796 -0.4125 -0.2668" rpy="0.03155910360450854 0.00996866505764844 0.7429270934423268"/> CHNAGING THIS ON WEDNESDAY SEP 11 -->
+        <!-- <origin xyz="0.5725015 -0.4188297 -0.2629327" rpy="0.0096794 -0.0028546 0.7357978"/> CORRECT VALUE OBTAINED AFTER POSE 2 KUKA -->
+        <!-- <origin xyz="0.1191248 -0.1369534 -0.0014446" rpy="0.0017781 -0.0007357 -0.7348171"/> -->
+        <!-- <origin xyz="0.5775893 -0.4121741 -0.265291" rpy="0.0150255 -0.0146531 0.7451824"/> -->
+        <origin xyz="0.5754642 -0.4159573 -0.2617773" rpy="0.0046846 -0.0042898 0.7420555"/>
+        <!-- <origin xyz="0 0 0" rpy="0 0 0 "/> -->
     </joint>
     <!-- iiwa -->
@@ -35,5 +42,5 @@
         </inertial>
         <visual>
-            <origin rpy="1.57 0 1.57" xyz="-0.0925 0 0.035" />
+            <origin rpy="1.57 0 1.57" xyz="-0.0925 0 0" />
             <geometry>
                 <mesh filename="package://lbr_description/meshes/iiwa7/collision/robotiq_gripper.stl" scale="0.001 0.001 0.001"/>
@@ -41,5 +48,5 @@
         </visual>
         <collision>
-            <origin rpy="1.57 0 1.57" xyz="-0.0925 0 0.035" />
+            <origin rpy="1.57 0 1.57" xyz="-0.0925 0 0" />
             <geometry>
                 <mesh filename="package://lbr_description/meshes/iiwa7/collision/robotiq_gripper.stl" scale="0.001 0.001 0.001"/>
@@ -50,5 +57,5 @@
         <parent link="link_7"/>
         <child link="link_ee"/>
-        <origin rpy="0 0 0" xyz="0 0 0"/>
+        <origin rpy="0 0 0" xyz="0 0 0.035"/>
     </joint>
     <link name="link_tcp"/>
@@ -56,5 +63,6 @@
         <parent link="link_ee"/>
         <child link="link_tcp"/>
-        <origin rpy="0 0 0" xyz="-0.00022 0.00163 0.17048"/>
+        <!-- <origin rpy="0 0 0" xyz="-0.00022 0.00163 0.17048"/> -->
+        <origin rpy="0 0 0" xyz="0.00031 0.00073 0.17152"/>
     </joint>
 </robot>

File: src/lbr_fri_ros2_stack/lbr_description/urdf/kuka_green/kuka_green.xacro (robot description, xacro)
@@ -19,5 +19,8 @@
         <!-- <origin xyz="0.8 0.7 -0.425" rpy="0 0 -2.356"/> -->
         <!-- <origin xyz="0.8 0.7 -0.47" rpy="0 0 -2.356"/> -->
-        <origin xyz="0.85 0.60 -0.46" rpy="0 0 -2.356"/>
+        <!-- <origin xyz="0.85 0.60 -0.46" rpy="0 0 -2.356"/> Friday-->
+        <!-- <origin xyz="0 0 0" rpy="0 0 0"/> -->
+        <!-- <origin xyz="0.8057409 0.6804944 -0.4295127" rpy="-0.0265684 0.0060622 -2.3834002"/> -->
+        <origin xyz="0.7947345 0.694259 -0.4280015" rpy="-0.0227401 0.0105353 -2.3640002"/>
     </joint>
     <!-- iiwa -->
@@ -56,5 +59,4 @@
         <parent link="link_ee"/>
         <child link="link_tcp"/>
-        <!-- <origin rpy="0 0 0" xyz="0.00051 -0.00012 0.23332"/> -->
         <origin rpy="0 0 0" xyz="0.00051 -0.00012 0.23332"/>
     </joint>

Commit message: before MSEC 1 week

File: src/lbr_fri_ros2_stack/lbr_description/urdf/kuka_blue/kuka_blue.xacro (robot description, xacro)
@@ -26,5 +26,12 @@
         <!-- <origin xyz="0.1191248 -0.1369534 -0.0014446" rpy="0.0017781 -0.0007357 -0.7348171"/> -->
         <!-- <origin xyz="0.5775893 -0.4121741 -0.265291" rpy="0.0150255 -0.0146531 0.7451824"/> -->
-        <origin xyz="0.5754642 -0.4159573 -0.2617773" rpy="0.0046846 -0.0042898 0.7420555"/>
+        <!-- RS_original -->
+        <!-- <origin xyz="0.5754642 -0.4159573 -0.2617773" rpy="0.0046846 -0.0042898 0.7420555"/>  -->
+        <!-- Sam 1cm forward in x edge3-->
+        <!-- <origin xyz="0.5654642 -0.4159573 -0.2717773" rpy="0.0046846 -0.0042898 0.7420555"/>  -->
+        <!-- PlayBack -->
+        <origin xyz="0.5754642 -0.4159573 -0.2417773" rpy="0.0046846 -0.0042898 0.7420555"/>
+        <!-- Sam 0.5cm forward in x -->
+        <!-- <origin xyz="0.5704642 -0.4159573 -0.2667773" rpy="0.0046846 -0.0042898 0.7420555"/>  -->
         <!-- <origin xyz="0 0 0" rpy="0 0 0 "/> -->
     </joint>
@@ -63,6 +70,10 @@
         <parent link="link_ee"/>
         <child link="link_tcp"/>
-        <!-- <origin rpy="0 0 0" xyz="-0.00022 0.00163 0.17048"/> -->
+        <!-- RS_Original -->
         <origin rpy="0 0 0" xyz="0.00031 0.00073 0.17152"/>
+        <!-- Sam 1cm backward in z -->
+        <!-- <origin rpy="0 0 0" xyz="0.00031 0.00073 0.16152"/> -->
+        <!-- Sam 0.5cm forward in z -->
+        <!-- <origin rpy="0 0 0" xyz="0.00031 0.00073 0.17652"/> -->
     </joint>
 </robot>

File: src/lbr_fri_ros2_stack/lbr_description/urdf/kuka_green/kuka_green.xacro (robot description, xacro)
@@ -22,7 +22,17 @@
         <!-- <origin xyz="0 0 0" rpy="0 0 0"/> -->
         <!-- <origin xyz="0.8057409 0.6804944 -0.4295127" rpy="-0.0265684 0.0060622 -2.3834002"/> -->
-        <!-- <origin xyz="0.7947345 0.694259 -0.4280015" rpy="-0.0227401 0.0105353 -2.3640002"/> -->
-        <!-- <origin xyz="0.7947345 0.694259 -0.4480015" rpy="-0.0227401 0.0105353 -2.3640002"/>  Friday -->
-        <origin xyz="0.7947345 0.694259 -0.4580015" rpy="-0.0227401 0.0105353 -2.3640002"/>
+         <!--RSOriginal-->
+        <!-- <origin xyz="0.7947345 0.694259 -0.4280015" rpy="-0.0227401 0.0105353 -2.3640002"/>   -->
+        <!-- <origin xyz="0.7947345 0.694259 -0.4330015" rpy="-0.0227401 0.0105353 -2.3640002"/> -->
+        <!--SAM 2cm below -->
+        <origin xyz="0.7947345 0.694259 -0.4480015" rpy="-0.0227401 0.0105353 -2.3640002"/>
+        <!-- PlayBack -->
+        <!-- <origin xyz="0.7947345 0.694259 -0.4530015" rpy="-0.0227401 0.0105353 -2.3640002"/> -->
+        <!-- ft_20_edge3 .... 28.5 deg -->
+        <!-- <origin xyz="0.8147345 0.694259 -0.4580015" rpy="-0.0227401 0.0105353 -2.3640002"/> -->
+        <!--SAM 3cm below -->
+        <!-- <origin xyz="0.7947345 0.694259 -0.4580015" rpy="-0.0227401 0.0105353 -2.3640002"/> -->
+        <!--SAM 4cm below -->
+        <!-- <origin xyz="0.7947345 0.694259 -0.4680015" rpy="-0.0227401 0.0105353 -2.3640002"/> -->
     </joint>
     <!-- iiwa -->

Commit message: after white xps stopped working

File: src/lbr_fri_ros2_stack/lbr_description/urdf/kuka_blue/kuka_blue.xacro (robot description, xacro)
@@ -71,5 +71,6 @@
         <child link="link_tcp"/>
         <!-- RS_Original -->
-        <origin rpy="0 0 0" xyz="0.00031 0.00073 0.17152"/>
+        <!-- <origin rpy="0 0 0" xyz="0.00031 0.00073 0.17152"/> --> <!-- original value used for robotiq gripper on chiseling project-->
+        <origin rpy="0 0 0" xyz="0.0688 -0.001 0.3506"/> <!-- UMI gripper data-->
         <!-- Sam 1cm backward in z -->
         <!-- <origin rpy="0 0 0" xyz="0.00031 0.00073 0.16152"/> -->

Commit message: created_tmp_msec for fusing files

File: src/lbr_fri_ros2_stack/lbr_description/urdf/kuka_blue/kuka_blue.xacro (robot description, xacro)
@@ -31,8 +31,10 @@
         <!-- <origin xyz="0.5654642 -0.4159573 -0.2717773" rpy="0.0046846 -0.0042898 0.7420555"/>  -->
         <!-- PlayBack -->
-        <origin xyz="0.5754642 -0.4159573 -0.2417773" rpy="0.0046846 -0.0042898 0.7420555"/>
+        <!-- <origin xyz="0.5754642 -0.4159573 -0.2417773" rpy="0.0046846 -0.0042898 0.7420555"/>  -->
         <!-- Sam 0.5cm forward in x -->
         <!-- <origin xyz="0.5704642 -0.4159573 -0.2667773" rpy="0.0046846 -0.0042898 0.7420555"/>  -->
         <!-- <origin xyz="0 0 0" rpy="0 0 0 "/> -->
+        <!-- original -->
+        <origin xyz="0.5754642 -0.4159573 -0.2417773" rpy="0.0 0.0 0.0"/>
     </joint>
     <!-- iiwa -->
@@ -71,5 +73,6 @@
         <child link="link_tcp"/>
         <!-- RS_Original -->
-        <origin rpy="0 0 0" xyz="0.00031 0.00073 0.17152"/>
+        <!-- <origin rpy="0 0 0" xyz="0.00031 0.00073 0.17152"/> --> <!-- original value used for robotiq gripper on chiseling project-->
+        <origin rpy="0 0 0" xyz="0.0688 -0.001 0.3506"/> <!-- UMI gripper data-->
         <!-- Sam 1cm backward in z -->
         <!-- <origin rpy="0 0 0" xyz="0.00031 0.00073 0.16152"/> -->

File: src/lbr_fri_ros2_stack/lbr_description/urdf/kuka_green/kuka_green.xacro (robot description, xacro)
@@ -25,5 +25,5 @@
         <!-- <origin xyz="0.7947345 0.694259 -0.4280015" rpy="-0.0227401 0.0105353 -2.3640002"/>   -->
         <!-- <origin xyz="0.7947345 0.694259 -0.4330015" rpy="-0.0227401 0.0105353 -2.3640002"/> -->
-        <!--SAM 2cm below -->
+        <!--SAM 2cm below BEFORE ANY CHANGES-->
         <origin xyz="0.7947345 0.694259 -0.4480015" rpy="-0.0227401 0.0105353 -2.3640002"/>
         <!-- PlayBack -->

Commit message: started working again --> add motive start stop recording functionality to service.launch.py

File: src/lbr_fri_ros2_stack/lbr_description/urdf/kuka_blue/kuka_blue.xacro (robot description, xacro)
@@ -46,18 +46,18 @@
     <link name="link_ee">
         <inertial>
-            <origin rpy="1.57 0 1.57" xyz="0 0 0.08524" />
+            <origin rpy="1.57 0 1.57" xyz="0 0 0.055525" />
             <mass value="0.55" />
             <inertia ixx="0.0001" ixy="0.0" ixz="0.0" iyy="0.0001" iyz="0.0" izz="0.0001" />
         </inertial>
         <visual>
-            <origin rpy="1.57 0 1.57" xyz="-0.0925 0 0" />
+            <origin rpy="1.57 0 1.57" xyz="0.0 0.0 0.0" />
             <geometry>
-                <mesh filename="package://lbr_description/meshes/iiwa7/collision/robotiq_gripper.stl" scale="0.001 0.001 0.001"/>
+                <mesh filename="package://lbr_description/meshes/iiwa7/visual/chisel.dae" scale="0.01 0.01 0.01"/>
             </geometry>
         </visual>
         <collision>
-            <origin rpy="1.57 0 1.57" xyz="-0.0925 0 0" />
+            <origin rpy="1.57 0 1.57" xyz="0.0 0.0 0.0" />
             <geometry>
-                <mesh filename="package://lbr_description/meshes/iiwa7/collision/robotiq_gripper.stl" scale="0.001 0.001 0.001"/>
+                <mesh filename="package://lbr_description/meshes/iiwa7/collision/chisel.stl" scale="0.001 0.001 0.001"/>
             </geometry>
         </collision>
@@ -66,17 +66,13 @@
         <parent link="link_7"/>
         <child link="link_ee"/>
-        <origin rpy="0 0 0" xyz="0 0 0.035"/>
+        <origin rpy="0 0 3.14" xyz="0 0 0.035"/>
     </joint>
+    <!-- TCP Link -->
     <link name="link_tcp"/>
     <joint name="joint_tcp" type="fixed">
         <parent link="link_ee"/>
         <child link="link_tcp"/>
-        <!-- RS_Original -->
-        <!-- <origin rpy="0 0 0" xyz="0.00031 0.00073 0.17152"/> --> <!-- original value used for robotiq gripper on chiseling project-->
-        <origin rpy="0 0 0" xyz="0.0688 -0.001 0.3506"/> <!-- UMI gripper data-->
-        <!-- Sam 1cm backward in z -->
-        <!-- <origin rpy="0 0 0" xyz="0.00031 0.00073 0.16152"/> -->
-        <!-- Sam 0.5cm forward in z -->
-        <!-- <origin rpy="0 0 0" xyz="0.00031 0.00073 0.17652"/> -->
+        <!-- <origin rpy="0 0 0" xyz="0.00051 -0.00012 0.23332"/> NO FORCE TOOL -->
+        <origin rpy="0 0 0" xyz="0.00243 0.0003 0.22498"/>
     </joint>
 </robot>

File: src/lbr_fri_ros2_stack/lbr_description/urdf/kuka_green/kuka_green.xacro (robot description, xacro)
@@ -44,18 +44,18 @@
     <link name="link_ee">
         <inertial>
-            <origin rpy="1.57 0 1.57" xyz="0 0 0.055525" />
+            <origin rpy="1.57 0 1.57" xyz="0 0 0.08524" />
             <mass value="0.55" />
             <inertia ixx="0.0001" ixy="0.0" ixz="0.0" iyy="0.0001" iyz="0.0" izz="0.0001" />
         </inertial>
         <visual>
-            <origin rpy="1.57 0 1.57" xyz="0.0 0.0 0.0" />
+            <origin rpy="1.57 0 1.57" xyz="-0.0925 0 0" />
             <geometry>
-                <mesh filename="package://lbr_description/meshes/iiwa7/visual/chisel.dae" scale="0.01 0.01 0.01"/>
+                <mesh filename="package://lbr_description/meshes/iiwa7/collision/robotiq_gripper.stl" scale="0.001 0.001 0.001"/>
             </geometry>
         </visual>
         <collision>
-            <origin rpy="1.57 0 1.57" xyz="0.0 0.0 0.0" />
+            <origin rpy="1.57 0 1.57" xyz="-0.0925 0 0" />
             <geometry>
-                <mesh filename="package://lbr_description/meshes/iiwa7/collision/chisel.stl" scale="0.001 0.001 0.001"/>
+                <mesh filename="package://lbr_description/meshes/iiwa7/collision/robotiq_gripper.stl" scale="0.001 0.001 0.001"/>
             </geometry>
         </collision>
@@ -64,13 +64,17 @@
         <parent link="link_7"/>
         <child link="link_ee"/>
-        <origin rpy="0 0 3.14" xyz="0 0 0.035"/>
+        <origin rpy="0 0 0" xyz="0 0 0.035"/>
     </joint>
-    <!-- TCP Link -->
     <link name="link_tcp"/>
     <joint name="joint_tcp" type="fixed">
         <parent link="link_ee"/>
         <child link="link_tcp"/>
-        <!-- <origin rpy="0 0 0" xyz="0.00051 -0.00012 0.23332"/> NO FORCE TOOL -->
-        <origin rpy="0 0 0" xyz="0.00243 0.0003 0.22498"/>
+        <!-- RS_Original -->
+        <!-- <origin rpy="0 0 0" xyz="0.00031 0.00073 0.17152"/> --> <!-- original value used for robotiq gripper on chiseling project-->
+        <origin rpy="0 0 0" xyz="0.0688 -0.001 0.3506"/> <!-- UMI gripper data-->
+        <!-- Sam 1cm backward in z -->
+        <!-- <origin rpy="0 0 0" xyz="0.00031 0.00073 0.16152"/> -->
+        <!-- Sam 0.5cm forward in z -->
+        <!-- <origin rpy="0 0 0" xyz="0.00031 0.00073 0.17652"/> -->
     </joint>
 </robot>

Commit message: added gripper aniket

File: src/lbr_fri_ros2_stack/lbr_description/urdf/kuka_blue/kuka_blue.xacro (robot description, xacro)
@@ -51,13 +51,13 @@
         </inertial>
         <visual>
-            <origin rpy="1.57 0 1.57" xyz="0.0 0.0 0.0" />
+            <origin rpy="0 3.14 0" xyz="0.0 0.0 0.0" />
             <geometry>
-                <mesh filename="package://lbr_description/meshes/iiwa7/visual/chisel.dae" scale="0.01 0.01 0.01"/>
+                <mesh filename="package://lbr_description/meshes/iiwa7/visual/aniket_gripper.dae" scale="0.001 0.001 0.001"/>
             </geometry>
         </visual>
         <collision>
-            <origin rpy="1.57 0 1.57" xyz="0.0 0.0 0.0" />
+            <origin rpy="0 3.14 0" xyz="0.0 0.0 0.0" />
             <geometry>
-                <mesh filename="package://lbr_description/meshes/iiwa7/collision/chisel.stl" scale="0.001 0.001 0.001"/>
+                <mesh filename="package://lbr_description/meshes/iiwa7/collision/aniket_gripper.stl" scale="0.001 0.001 0.001"/>
             </geometry>
         </collision>

Commit message: Refactor frame prefix logic and update robot pose
Updates the frame prefix configuration to use a cleaner Python expression for consistent path formatting.

Additionally, cleans up redundant commented-out code in the URDF and updates the tool center point (TCP) offset to the latest calibrated values.

File: src/lbr_fri_ros2_stack/lbr_description/urdf/kuka_blue/kuka_blue.xacro (robot description, xacro)
@@ -17,23 +17,4 @@
         <parent link="world" />
         <child link="link_0" />
-        <!-- <origin xyz="0.55 -0.4 -0.25" rpy="0 0 0.783"/> -->
-        <!-- <origin xyz="0.55 -0.4 -0.35" rpy="0 0 0.783"/> -->
-        <!-- <origin xyz="0.55 -0.4 -0.264" rpy="0 0 0.783"/>   CORRECT VALUE USED ON FRIDAY DEMO -->
-        <!-- <origin xyz="0.5796 -0.4125 -0.2668" rpy="0.74287 -0.01400 0.029986"/> RS -->
-        <!-- <origin xyz="0.5796 -0.4125 -0.2668" rpy="0.03155910360450854 0.00996866505764844 0.7429270934423268"/>  RS-->
-        <!-- <origin xyz="0.5796 -0.4125 -0.2668" rpy="0.03155910360450854 0.00996866505764844 0.7429270934423268"/> CHNAGING THIS ON WEDNESDAY SEP 11 -->
-        <!-- <origin xyz="0.5725015 -0.4188297 -0.2629327" rpy="0.0096794 -0.0028546 0.7357978"/> CORRECT VALUE OBTAINED AFTER POSE 2 KUKA -->
-        <!-- <origin xyz="0.1191248 -0.1369534 -0.0014446" rpy="0.0017781 -0.0007357 -0.7348171"/> -->
-        <!-- <origin xyz="0.5775893 -0.4121741 -0.265291" rpy="0.0150255 -0.0146531 0.7451824"/> -->
-        <!-- RS_original -->
-        <!-- <origin xyz="0.5754642 -0.4159573 -0.2617773" rpy="0.0046846 -0.0042898 0.7420555"/>  -->
-        <!-- Sam 1cm forward in x edge3-->
-        <!-- <origin xyz="0.5654642 -0.4159573 -0.2717773" rpy="0.0046846 -0.0042898 0.7420555"/>  -->
-        <!-- PlayBack -->
-        <!-- <origin xyz="0.5754642 -0.4159573 -0.2417773" rpy="0.0046846 -0.0042898 0.7420555"/>  -->
-        <!-- Sam 0.5cm forward in x -->
-        <!-- <origin xyz="0.5704642 -0.4159573 -0.2667773" rpy="0.0046846 -0.0042898 0.7420555"/>  -->
-        <!-- <origin xyz="0 0 0" rpy="0 0 0 "/> -->
-        <!-- original -->
         <origin xyz="0.5754642 -0.4159573 -0.2417773" rpy="0.0 0.0 0.0"/>
     </joint>
@@ -74,5 +55,6 @@
         <child link="link_tcp"/>
         <!-- <origin rpy="0 0 0" xyz="0.00051 -0.00012 0.23332"/> NO FORCE TOOL -->
-        <origin rpy="0 0 0" xyz="0.00243 0.0003 0.22498"/>
+        <!-- <origin rpy="0 0 0" xyz="0.00243 0.0003 0.22498"/> -->
+        <origin rpy="0 0 0" xyz="0.0 0.0 0.33149"/>
     </joint>
 </robot>

Commit message: Modularize LBR description and control stack
Refactor the LBR description and control logic into modular XACRO files to improve maintainability and support flexible robot configurations.

This update introduces dedicated macros for Gazebo integration and system interfaces, allowing for a cleaner separation between simulation and hardware-specific configurations.

File: src/lbr_fri_ros2_stack/lbr_description/urdf/kuka_blue/kuka_blue.xacro (robot description, xacro)
@@ -3,7 +3,6 @@
 <robot name="iiwa7" xmlns:xacro="http://www.ros.org/wiki/xacro">
     <!-- include the lbr iiwa macro -->
-    <xacro:include filename="$(find lbr_description)/urdf/iiwa7/iiwa7_description.xacro" />
-    <xacro:include filename="$(find robotiq_description)/urdf/robotiq_2f_85_macro.urdf.xacro" />
-    <xacro:arg name="robot_name" default="lbr" />
+    <xacro:include filename="$(find lbr_description)/urdf/iiwa7/iiwa7_description_mod.xacro" />
+    <!-- <xacro:include filename="$(find robotiq_description)/urdf/robotiq_2f_85_macro.urdf.xacro" /> -->
     <xacro:arg name="sim" default="true" />
     <xacro:arg name="use_fake_hardware" default="true" />
@@ -12,16 +11,16 @@
         default="$(find lbr_ros2_control)/config/lbr_system_parameters.yaml" />
     <!-- fixed to world, see http://classic.gazebosim.org/tutorials?tut=ros_urdf&cat=connect_ros -->
-    <link name="world" />
-    <!-- joint between world and link_0 -->
-    <joint name="world_joint" type="fixed">
-        <parent link="world" />
-        <child link="link_0" />
-        <origin xyz="0.5754642 -0.4159573 -0.2417773" rpy="0.0 0.0 0.0"/>
-    </joint>
+    <link name="world">
+        <origin xyz="0 0 0" rpy="0 0 0"/>
+    </link>
+    <xacro:arg name="robot_name" default="kuka_blue" />
     <!-- iiwa -->
     <xacro:iiwa7
         robot_name="$(arg robot_name)"
+        parent = "world"
         sim="$(arg sim)"
         system_parameters_path="$(arg system_parameters_path)" />
+        <origin xyz="0 0 0" rpy="0 0 0"/>
+    </xacro:iiwa7>
     <!-- End Effector -->
     <link name="link_ee">
