Commit message: refactor

File: src/lbr_fri_ros2_stack/lbr_moveit_config/kuka_blue_moveit_config/config/iiwa7.ros2_control.xacro (robot description, xacro)
@@ -8,50 +8,50 @@
                 <plugin>mock_components/GenericSystem</plugin>
             </hardware>
-            <joint name="A1">
+            <joint name="kuka_blue_A1">
                 <command_interface name="position"/>
                 <state_interface name="position">
-                  <param name="initial_value">${initial_positions['A1']}</param>
+                  <param name="initial_value">${initial_positions['kuka_blue_A1']}</param>
                 </state_interface>
                 <state_interface name="velocity"/>
             </joint>
-            <joint name="A2">
+            <joint name="kuka_blue_A2">
                 <command_interface name="position"/>
                 <state_interface name="position">
-                  <param name="initial_value">${initial_positions['A2']}</param>
+                  <param name="initial_value">${initial_positions['kuka_blue_A2']}</param>
                 </state_interface>
                 <state_interface name="velocity"/>
             </joint>
-            <joint name="A3">
+            <joint name="kuka_blue_A3">
                 <command_interface name="position"/>
                 <state_interface name="position">
-                  <param name="initial_value">${initial_positions['A3']}</param>
+                  <param name="initial_value">${initial_positions['kuka_blue_A3']}</param>
                 </state_interface>
                 <state_interface name="velocity"/>
             </joint>
-            <joint name="A4">
+            <joint name="kuka_blue_A4">
                 <command_interface name="position"/>
                 <state_interface name="position">
-                  <param name="initial_value">${initial_positions['A4']}</param>
+                  <param name="initial_value">${initial_positions['kuka_blue_A4']}</param>
                 </state_interface>
                 <state_interface name="velocity"/>
             </joint>
-            <joint name="A5">
+            <joint name="kuka_blue_A5">
                 <command_interface name="position"/>
                 <state_interface name="position">
-                  <param name="initial_value">${initial_positions['A5']}</param>
+                  <param name="initial_value">${initial_positions['kuka_blue_A5']}</param>
                 </state_interface>
                 <state_interface name="velocity"/>
             </joint>
-            <joint name="A6">
+            <joint name="kuka_blue_A6">
                 <command_interface name="position"/>
                 <state_interface name="position">
-                  <param name="initial_value">${initial_positions['A6']}</param>
+                  <param name="initial_value">${initial_positions['kuka_blue_A6']}</param>
                 </state_interface>
                 <state_interface name="velocity"/>
             </joint>
-            <joint name="A7">
+            <joint name="kuka_blue_A7">
                 <command_interface name="position"/>
                 <state_interface name="position">
-                  <param name="initial_value">${initial_positions['A7']}</param>
+                  <param name="initial_value">${initial_positions['kuka_blue_A7']}</param>
                 </state_interface>
                 <state_interface name="velocity"/>

File: src/lbr_fri_ros2_stack/lbr_ros2_control/config/lbr_system_interface_mod.xacro (robot description, xacro)
@@ -16,4 +16,6 @@
                 <hardware>
                     <plugin>lbr_ros2_control::SystemInterface</plugin>
+                    <param name="fri_client_sdk_major_version">${system_parameters['hardware']['fri_client_sdk']['major_version']}</param>
+                    <param name="fri_client_sdk_minor_version">${system_parameters['hardware']['fri_client_sdk']['minor_version']}</param>
                     <param name="client_command_mode">${system_parameters['hardware']['client_command_mode']}</param>
                     <param name="port_id">${system_parameters['hardware'].get(robot_name + '_port_id', system_parameters['hardware']['port_id'])}</param>
