Commit message: Automate controller configuration generation
Improves launch flexibility by dynamically generating controller configurations based on the loaded robot description. This replaces static, hard-coded YAML configurations with an automated process that extracts joint names and sensor frames directly from the URDF.

Adds support for configurable description variants and moveit packages across all launch files to simplify handling of different robot models and custom configurations.

File: src/lbr_fri_ros2_stack/lbr_description/gazebo/green_gazebo.xacro (robot description, xacro)
@@ -1,9 +1,11 @@
 <?xml version="1.0"?>
 <robot xmlns:xacro="http://www.ros.org/wiki/xacro">
-    <xacro:macro name="lbr_gazebo" params="robot_name:=^|green">
+    <xacro:macro
+        name="lbr_gazebo"
+        params="robot_name:=^|green controllers_path:=^|'$(find lbr_ros2_control)/config/lbr_controllers.yaml'">
         <!-- ros_control-plugin -->
         <gazebo>
             <plugin name="gazebo_ros2_control" filename="libgazebo_ros2_control.so">
-                <parameters>$(find lbr_ros2_control)/config/lbr_controllers.yaml</parameters>
+                <parameters>${controllers_path}</parameters>
                 <ros>
                     <namespace>/${robot_name}</namespace>

File: src/lbr_fri_ros2_stack/lbr_description/gazebo/lbr_gazebo.xacro (robot description, xacro)
@@ -1,9 +1,11 @@
 <?xml version="1.0"?>
 <robot xmlns:xacro="http://www.ros.org/wiki/xacro">
-    <xacro:macro name="lbr_gazebo" params="robot_name:=^|lbr">
+    <xacro:macro
+        name="lbr_gazebo"
+        params="robot_name:=^|lbr controllers_path:=^|'$(find lbr_ros2_control)/config/lbr_controllers.yaml'">
         <!-- ros_control-plugin -->
         <gazebo>
             <plugin name="gazebo_ros2_control" filename="libgazebo_ros2_control.so">
-                <parameters>$(find lbr_ros2_control)/config/lbr_controllers.yaml</parameters>
+                <parameters>${controllers_path}</parameters>
                 <ros>
                     <namespace>/${robot_name}</namespace>

File: src/lbr_fri_ros2_stack/lbr_description/gazebo/lbr_gazebo_mod.xacro (robot description, xacro)
@@ -1,9 +1,11 @@
 <?xml version="1.0"?>
 <robot xmlns:xacro="http://www.ros.org/wiki/xacro">
-    <xacro:macro name="lbr_gazebo" params="robot_name:=^|kuka_blue">
+    <xacro:macro
+        name="lbr_gazebo"
+        params="robot_name:=^|lbr controllers_path:=^|'$(find lbr_ros2_control)/config/lbr_controllers.yaml'">
         <!-- ros_control-plugin -->
         <gazebo>
             <plugin name="gazebo_ros2_control" filename="libgazebo_ros2_control.so">
-                <parameters>$(find lbr_ros2_control)/config/lbr_controllers.yaml</parameters>
+                <parameters>${controllers_path}</parameters>
                 <ros>
                     <namespace>/${robot_name}</namespace>

File: src/lbr_fri_ros2_stack/lbr_description/urdf/green/green.xacro (robot description, xacro)
@@ -9,4 +9,7 @@
         name="system_parameters_path"
         default="$(find lbr_ros2_control)/config/lbr_system_parameters.yaml" />
+    <xacro:arg
+        name="controllers_path"
+        default="$(find lbr_ros2_control)/config/lbr_controllers.yaml" />
     <!-- fixed to world, see http://classic.gazebosim.org/tutorials?tut=ros_urdf&cat=connect_ros -->
     <link name="world" />
@@ -21,4 +24,5 @@
         robot_name="$(arg robot_name)"
         sim="$(arg sim)"
-        system_parameters_path="$(arg system_parameters_path)" />
+        system_parameters_path="$(arg system_parameters_path)"
+        controllers_path="$(arg controllers_path)" />
 </robot>

File: src/lbr_fri_ros2_stack/lbr_description/urdf/green/green_description.xacro (robot description, xacro)
@@ -3,5 +3,5 @@
     <!-- robot as extracted via https://github.com/syuntoku14/fusion2urdf -->
     <xacro:macro name="iiwa7"
-        params="robot_name:=^|green sim:=^=true system_parameters_path:=^|'$(find lbr_ros2_control)/config/lbr_system_parameters.yaml'">
+        params="robot_name:=^|green sim:=^=true system_parameters_path:=^|'$(find lbr_ros2_control)/config/lbr_system_parameters.yaml' controllers_path:=^|'$(find lbr_ros2_control)/config/lbr_controllers.yaml'">
         <!-- includes -->
         <xacro:include filename="$(find lbr_description)/gazebo/green_gazebo.xacro" />
@@ -16,5 +16,5 @@
         <xacro:property name="joint_friction" value="0.1" />
         <!-- macros for simulation and real hardware -->
-        <xacro:lbr_gazebo robot_name="${robot_name}" />
+        <xacro:lbr_gazebo robot_name="${robot_name}" controllers_path="${controllers_path}" />
         <xacro:lbr_system_interface
             sim="${sim}"

File: src/lbr_fri_ros2_stack/lbr_description/urdf/iiwa14/iiwa14.xacro (robot description, xacro)
@@ -9,4 +9,7 @@
         name="system_parameters_path"
         default="$(find lbr_ros2_control)/config/lbr_system_parameters.yaml" />
+    <xacro:arg
+        name="controllers_path"
+        default="$(find lbr_ros2_control)/config/lbr_controllers.yaml" />
     <!-- fixed to world, see http://classic.gazebosim.org/tutorials?tut=ros_urdf&cat=connect_ros -->
     <link name="world" />
@@ -21,4 +24,5 @@
         robot_name="$(arg robot_name)"
         sim="$(arg sim)"
-        system_parameters_path="$(arg system_parameters_path)" />
+        system_parameters_path="$(arg system_parameters_path)"
+        controllers_path="$(arg controllers_path)" />
 </robot>

File: src/lbr_fri_ros2_stack/lbr_description/urdf/iiwa14/iiwa14_description.xacro (robot description, xacro)
@@ -3,5 +3,5 @@
     <!-- robot as extracted via https://github.com/syuntoku14/fusion2urdf -->
     <xacro:macro name="iiwa14"
-        params="robot_name:=^|lbr sim:=^=true system_parameters_path:=^|'$(find lbr_ros2_control)/config/lbr_system_parameters.yaml'">
+        params="robot_name:=^|lbr sim:=^=true system_parameters_path:=^|'$(find lbr_ros2_control)/config/lbr_system_parameters.yaml' controllers_path:=^|'$(find lbr_ros2_control)/config/lbr_controllers.yaml'">
         <!-- includes -->
         <xacro:include filename="$(find lbr_description)/gazebo/lbr_gazebo.xacro" />
@@ -16,5 +16,5 @@
         <xacro:property name="joint_friction" value="0.1" />
         <!-- macros for simulation and real hardware -->
-        <xacro:lbr_gazebo robot_name="${robot_name}" />
+        <xacro:lbr_gazebo robot_name="${robot_name}" controllers_path="${controllers_path}" />
         <xacro:lbr_system_interface
             sim="${sim}"

File: src/lbr_fri_ros2_stack/lbr_description/urdf/iiwa7/iiwa7.xacro (robot description, xacro)
@@ -9,4 +9,7 @@
         name="system_parameters_path"
         default="$(find lbr_ros2_control)/config/lbr_system_parameters.yaml" />
+    <xacro:arg
+        name="controllers_path"
+        default="$(find lbr_ros2_control)/config/lbr_controllers.yaml" />
     <!-- fixed to world, see http://classic.gazebosim.org/tutorials?tut=ros_urdf&cat=connect_ros -->
     <link name="world" />
@@ -21,4 +24,5 @@
         robot_name="$(arg robot_name)"
         sim="$(arg sim)"
-        system_parameters_path="$(arg system_parameters_path)" />
+        system_parameters_path="$(arg system_parameters_path)"
+        controllers_path="$(arg controllers_path)" />
 </robot>

File: src/lbr_fri_ros2_stack/lbr_description/urdf/iiwa7/iiwa7_description.xacro (robot description, xacro)
@@ -3,5 +3,5 @@
     <!-- robot as extracted via https://github.com/syuntoku14/fusion2urdf -->
     <xacro:macro name="iiwa7"
-        params="robot_name:=^|lbr sim:=^=true system_parameters_path:=^|'$(find lbr_ros2_control)/config/lbr_system_parameters.yaml'">
+        params="robot_name:=^|lbr sim:=^=true system_parameters_path:=^|'$(find lbr_ros2_control)/config/lbr_system_parameters.yaml' controllers_path:=^|'$(find lbr_ros2_control)/config/lbr_controllers.yaml'">
         <!-- includes -->
         <xacro:include filename="$(find lbr_description)/gazebo/lbr_gazebo.xacro" />
@@ -16,5 +16,5 @@
         <xacro:property name="joint_friction" value="0.1" />
         <!-- macros for simulation and real hardware -->
-        <xacro:lbr_gazebo robot_name="${robot_name}" />
+        <xacro:lbr_gazebo robot_name="${robot_name}" controllers_path="${controllers_path}" />
         <xacro:lbr_system_interface
             sim="${sim}"

File: src/lbr_fri_ros2_stack/lbr_description/urdf/iiwa7/iiwa7_description_mod.xacro (robot description, xacro)
@@ -3,5 +3,5 @@
     <!-- robot as extracted via https://github.com/syuntoku14/fusion2urdf -->
     <xacro:macro name="iiwa7"
-        params="robot_name:=^|lbr sim:=^=true system_parameters_path:=^|'$(find lbr_ros2_control)/config/lbr_system_parameters.yaml'">
+        params="robot_name:=^|lbr sim:=^=true system_parameters_path:=^|'$(find lbr_ros2_control)/config/lbr_system_parameters.yaml' controllers_path:=^|'$(find lbr_ros2_control)/config/lbr_controllers.yaml'">
         <!-- includes -->
         <xacro:include filename="$(find lbr_description)/gazebo/lbr_gazebo_mod.xacro" />
@@ -28,5 +28,5 @@
         <xacro:property name="joint_friction" value="0.1" />
         <!-- macros for simulation and real hardware -->
-        <xacro:lbr_gazebo robot_name="${robot_name}" />
+        <xacro:lbr_gazebo robot_name="${robot_name}" controllers_path="${controllers_path}" />
         <xacro:lbr_system_interface
             sim="${sim}"

File: src/lbr_fri_ros2_stack/lbr_description/urdf/iiwa7/iiwa7_kuka_blue.xacro (robot description, xacro)
@@ -9,4 +9,7 @@
         name="system_parameters_path"
         default="$(find lbr_ros2_control)/config/lbr_system_parameters.yaml" />
+    <xacro:arg
+        name="controllers_path"
+        default="$(find lbr_ros2_control)/config/lbr_controllers.yaml" />
     <!-- fixed to world, see http://classic.gazebosim.org/tutorials?tut=ros_urdf&cat=connect_ros -->
     <link name="world" />
@@ -22,4 +25,5 @@
         robot_name="$(arg robot_name)"
         sim="$(arg sim)"
-        system_parameters_path="$(arg system_parameters_path)" />
+        system_parameters_path="$(arg system_parameters_path)"
+        controllers_path="$(arg controllers_path)" />
 </robot>

File: src/lbr_fri_ros2_stack/lbr_description/urdf/iiwa7/iiwa7_mod.xacro (robot description, xacro)
@@ -9,4 +9,7 @@
         name="system_parameters_path"
         default="$(find lbr_ros2_control)/config/lbr_system_parameters.yaml" />
+    <xacro:arg
+        name="controllers_path"
+        default="$(find lbr_ros2_control)/config/lbr_controllers.yaml" />
     <!-- fixed to world, see http://classic.gazebosim.org/tutorials?tut=ros_urdf&cat=connect_ros -->
     <link name="world" />
@@ -21,4 +24,5 @@
         robot_name="$(arg robot_name)"
         sim="$(arg sim)"
-        system_parameters_path="$(arg system_parameters_path)" />
+        system_parameters_path="$(arg system_parameters_path)"
+        controllers_path="$(arg controllers_path)" />
 </robot>

File: src/lbr_fri_ros2_stack/lbr_description/urdf/kuka_blue/kuka_blue.xacro (robot description, xacro)
@@ -9,4 +9,7 @@
         name="system_parameters_path"
         default="$(find lbr_ros2_control)/config/lbr_system_parameters.yaml" />
+    <xacro:arg
+        name="controllers_path"
+        default="$(find lbr_ros2_control)/config/lbr_controllers.yaml" />
     <xacro:arg name="robot_name" default="kuka_blue" />
     <xacro:property name="robot_prefix" value="$(arg robot_name)" />
@@ -22,5 +25,6 @@
         robot_name="$(arg robot_name)"
         sim="$(arg sim)"
-        system_parameters_path="$(arg system_parameters_path)" />
+        system_parameters_path="$(arg system_parameters_path)"
+        controllers_path="$(arg controllers_path)" />
     <!-- End Effector -->
     <link name="${robot_prefix}_link_ee">

File: src/lbr_fri_ros2_stack/lbr_description/urdf/kuka_green/kuka_green.xacro (robot description, xacro)
@@ -9,4 +9,7 @@
         name="system_parameters_path"
         default="$(find lbr_ros2_control)/config/lbr_system_parameters.yaml" />
+    <xacro:arg
+        name="controllers_path"
+        default="$(find lbr_ros2_control)/config/lbr_controllers.yaml" />
     <!-- fixed to world, see http://classic.gazebosim.org/tutorials?tut=ros_urdf&cat=connect_ros -->
     <link name="world" />
@@ -40,5 +43,6 @@
         robot_name="$(arg robot_name)"
         sim="$(arg sim)"
-        system_parameters_path="$(arg system_parameters_path)" />
+        system_parameters_path="$(arg system_parameters_path)"
+        controllers_path="$(arg controllers_path)" />
     <!-- End Effector -->
     <link name="link_ee">

File: src/lbr_fri_ros2_stack/lbr_description/urdf/med14/med14.xacro (robot description, xacro)
@@ -9,4 +9,7 @@
         name="system_parameters_path"
         default="$(find lbr_ros2_control)/config/lbr_system_parameters.yaml" />
+    <xacro:arg
+        name="controllers_path"
+        default="$(find lbr_ros2_control)/config/lbr_controllers.yaml" />
     <!-- fixed to world, see http://classic.gazebosim.org/tutorials?tut=ros_urdf&cat=connect_ros -->
     <link name="world" />
@@ -21,4 +24,5 @@
         robot_name="$(arg robot_name)"
         sim="$(arg sim)"
-        system_parameters_path="$(arg system_parameters_path)" />
+        system_parameters_path="$(arg system_parameters_path)"
+        controllers_path="$(arg controllers_path)" />
 </robot>

File: src/lbr_fri_ros2_stack/lbr_description/urdf/med14/med14_description.xacro (robot description, xacro)
@@ -3,5 +3,5 @@
     <!-- robot as extracted via https://github.com/syuntoku14/fusion2urdf -->
     <xacro:macro name="med14"
-        params="robot_name:=^|lbr sim:=^=true system_parameters_path:=^|'$(find lbr_ros2_control)/config/lbr_system_parameters.yaml'">
+        params="robot_name:=^|lbr sim:=^=true system_parameters_path:=^|'$(find lbr_ros2_control)/config/lbr_system_parameters.yaml' controllers_path:=^|'$(find lbr_ros2_control)/config/lbr_controllers.yaml'">
         <!-- includes -->
         <xacro:include filename="$(find lbr_description)/gazebo/lbr_gazebo.xacro" />
@@ -16,5 +16,5 @@
         <xacro:property name="joint_friction" value="0.1" />
         <!-- macros for simulation and real hardware -->
-        <xacro:lbr_gazebo robot_name="${robot_name}" />
+        <xacro:lbr_gazebo robot_name="${robot_name}" controllers_path="${controllers_path}" />
         <xacro:lbr_system_interface
             sim="${sim}"

File: src/lbr_fri_ros2_stack/lbr_description/urdf/med7/med7.xacro (robot description, xacro)
@@ -9,4 +9,7 @@
         name="system_parameters_path"
         default="$(find lbr_ros2_control)/config/lbr_system_parameters.yaml" />
+    <xacro:arg
+        name="controllers_path"
+        default="$(find lbr_ros2_control)/config/lbr_controllers.yaml" />
     <!-- fixed to world, see http://classic.gazebosim.org/tutorials?tut=ros_urdf&cat=connect_ros -->
     <link name="world" />
@@ -21,4 +24,5 @@
         robot_name="$(arg robot_name)"
         sim="$(arg sim)"
-        system_parameters_path="$(arg system_parameters_path)" />
+        system_parameters_path="$(arg system_parameters_path)"
+        controllers_path="$(arg controllers_path)" />
 </robot>

File: src/lbr_fri_ros2_stack/lbr_description/urdf/med7/med7_description.xacro (robot description, xacro)
@@ -3,5 +3,5 @@
     <!-- robot as extracted via https://github.com/syuntoku14/fusion2urdf -->
     <xacro:macro name="med7"
-        params="robot_name:=^|lbr sim:=^=true system_parameters_path:=^|'$(find lbr_ros2_control)/config/lbr_system_parameters.yaml'">
+        params="robot_name:=^|lbr sim:=^=true system_parameters_path:=^|'$(find lbr_ros2_control)/config/lbr_system_parameters.yaml' controllers_path:=^|'$(find lbr_ros2_control)/config/lbr_controllers.yaml'">
         <!-- includes -->
         <xacro:include filename="$(find lbr_description)/gazebo/lbr_gazebo.xacro" />
@@ -16,5 +16,5 @@
         <xacro:property name="joint_friction" value="0.1" />
         <!-- macros for simulation and real hardware -->
-        <xacro:lbr_gazebo robot_name="${robot_name}" />
+        <xacro:lbr_gazebo robot_name="${robot_name}" controllers_path="${controllers_path}" />
         <xacro:lbr_system_interface
             sim="${sim}"
