Commit message: refactor large -- remove mod file

File: src/lbr_fri_ros2_stack/lbr_description/gazebo/lbr_gazebo.xacro (robot description, xacro)
@@ -3,5 +3,11 @@
     <xacro:macro
         name="lbr_gazebo"
-        params="robot_name:=^|lbr controllers_path:=^|'$(find lbr_ros2_control)/config/lbr_controllers.yaml'">
+        params="robot_name:=^|lbr controllers_path:=^|'$(find lbr_ros2_control)/config/lbr_controllers.yaml' prefix_model_names:=^=false">
+        <xacro:property
+            name="use_prefix"
+            value="${str(prefix_model_names).lower() == 'true'}" />
+        <xacro:property
+            name="name_prefix"
+            value="${robot_name + '_' if use_prefix else ''}" />
         <!-- ros_control-plugin -->
         <gazebo>
@@ -29,19 +35,19 @@
         </xacro:macro>
         <!-- references -->
-        <xacro:gazebo_link_reference name="link_0" />
-        <xacro:gazebo_joint_reference name="A1" />
-        <xacro:gazebo_link_reference name="link_1" />
-        <xacro:gazebo_joint_reference name="A2" />
-        <xacro:gazebo_link_reference name="link_2" />
-        <xacro:gazebo_joint_reference name="A3" />
-        <xacro:gazebo_link_reference name="link_3" />
-        <xacro:gazebo_joint_reference name="A4" />
-        <xacro:gazebo_link_reference name="link_4" />
-        <xacro:gazebo_joint_reference name="A5" />
-        <xacro:gazebo_link_reference name="link_5" />
-        <xacro:gazebo_joint_reference name="A6" />
-        <xacro:gazebo_link_reference name="link_6" />
-        <xacro:gazebo_joint_reference name="A7" />
-        <xacro:gazebo_link_reference name="link_7" />
+        <xacro:gazebo_link_reference name="${name_prefix}link_0" />
+        <xacro:gazebo_joint_reference name="${name_prefix}A1" />
+        <xacro:gazebo_link_reference name="${name_prefix}link_1" />
+        <xacro:gazebo_joint_reference name="${name_prefix}A2" />
+        <xacro:gazebo_link_reference name="${name_prefix}link_2" />
+        <xacro:gazebo_joint_reference name="${name_prefix}A3" />
+        <xacro:gazebo_link_reference name="${name_prefix}link_3" />
+        <xacro:gazebo_joint_reference name="${name_prefix}A4" />
+        <xacro:gazebo_link_reference name="${name_prefix}link_4" />
+        <xacro:gazebo_joint_reference name="${name_prefix}A5" />
+        <xacro:gazebo_link_reference name="${name_prefix}link_5" />
+        <xacro:gazebo_joint_reference name="${name_prefix}A6" />
+        <xacro:gazebo_link_reference name="${name_prefix}link_6" />
+        <xacro:gazebo_joint_reference name="${name_prefix}A7" />
+        <xacro:gazebo_link_reference name="${name_prefix}link_7" />
     </xacro:macro>
 </robot>

File: src/lbr_fri_ros2_stack/lbr_description/urdf/iiwa7/iiwa7_description.xacro (robot description, xacro)
@@ -2,25 +2,64 @@
 <robot xmlns:xacro="http://www.ros.org/wiki/xacro">
     <!-- robot as extracted via https://github.com/syuntoku14/fusion2urdf -->
-    <xacro:macro name="iiwa7"
-        params="robot_name:=^|lbr sim:=^=true system_parameters_path:=^|'$(find lbr_ros2_control)/config/lbr_system_parameters.yaml' controllers_path:=^|'$(find lbr_ros2_control)/config/lbr_controllers.yaml'">
+    <xacro:macro
+        name="iiwa7"
+        params="robot_name:=^|lbr sim:=^=true system_parameters_path:=^|'$(find lbr_ros2_control)/config/lbr_system_parameters.yaml' controllers_path:=^|'$(find lbr_ros2_control)/config/lbr_controllers.yaml' prefix_model_names:=^=false">
         <!-- includes -->
         <xacro:include filename="$(find lbr_description)/gazebo/lbr_gazebo.xacro" />
         <xacro:include filename="$(find lbr_ros2_control)/config/lbr_system_interface.xacro" />
         <!-- joint limits via yaml -->
-        <xacro:property name="joint_limits_path"
+        <xacro:property
+            name="joint_limits_path"
             value="$(find lbr_description)/urdf/iiwa7/joint_limits.yaml" />
-        <xacro:property name="joint_limits" value="${xacro.load_yaml(joint_limits_path)}" />
+        <xacro:property name="base_joint_limits" value="${xacro.load_yaml(joint_limits_path)}" />
+        <xacro:property
+            name="use_prefix"
+            value="${str(prefix_model_names).lower() == 'true'}" />
+        <xacro:property
+            name="name_prefix"
+            value="${robot_name + '_' if use_prefix else ''}" />
+        <xacro:property
+            name="joint_limits"
+            value="${dict([
+                (name_prefix + 'A1', base_joint_limits['A1']),
+                (name_prefix + 'A2', base_joint_limits['A2']),
+                (name_prefix + 'A3', base_joint_limits['A3']),
+                (name_prefix + 'A4', base_joint_limits['A4']),
+                (name_prefix + 'A5', base_joint_limits['A5']),
+                (name_prefix + 'A6', base_joint_limits['A6']),
+                (name_prefix + 'A7', base_joint_limits['A7']),
+            ]) if use_prefix else base_joint_limits}" />
         <!-- constants -->
         <xacro:property name="PI" value="3.1415926535897931" />
         <xacro:property name="joint_damping" value="10.0" />
         <xacro:property name="joint_friction" value="0.1" />
+        <!-- canonical link and joint names -->
+        <xacro:property name="link_0_name" value="${name_prefix + 'link_0'}" />
+        <xacro:property name="link_1_name" value="${name_prefix + 'link_1'}" />
+        <xacro:property name="link_2_name" value="${name_prefix + 'link_2'}" />
+        <xacro:property name="link_3_name" value="${name_prefix + 'link_3'}" />
+        <xacro:property name="link_4_name" value="${name_prefix + 'link_4'}" />
+        <xacro:property name="link_5_name" value="${name_prefix + 'link_5'}" />
+        <xacro:property name="link_6_name" value="${name_prefix + 'link_6'}" />
+        <xacro:property name="link_7_name" value="${name_prefix + 'link_7'}" />
+        <xacro:property name="joint_a1_name" value="${name_prefix + 'A1'}" />
+        <xacro:property name="joint_a2_name" value="${name_prefix + 'A2'}" />
+        <xacro:property name="joint_a3_name" value="${name_prefix + 'A3'}" />
+        <xacro:property name="joint_a4_name" value="${name_prefix + 'A4'}" />
+        <xacro:property name="joint_a5_name" value="${name_prefix + 'A5'}" />
+        <xacro:property name="joint_a6_name" value="${name_prefix + 'A6'}" />
+        <xacro:property name="joint_a7_name" value="${name_prefix + 'A7'}" />
         <!-- macros for simulation and real hardware -->
-        <xacro:lbr_gazebo robot_name="${robot_name}" controllers_path="${controllers_path}" />
+        <xacro:lbr_gazebo
+            robot_name="${robot_name}"
+            controllers_path="${controllers_path}"
+            prefix_model_names="${use_prefix}" />
         <xacro:lbr_system_interface
             sim="${sim}"
             joint_limits="${joint_limits}"
             system_parameters_path="${system_parameters_path}"
-            robot_name="${robot_name}"/>
-        <link name="link_0">
+            robot_name="${robot_name}"
+            prefix_model_names="${use_prefix}" />
+        <link name="${link_0_name}">
             <inertial>
                 <origin rpy="0 0 0" xyz="-0.012857 0.0 0.069964" />
@@ -42,17 +81,17 @@
             </collision>
         </link>
-        <joint name="A1" type="revolute">
+        <joint name="${joint_a1_name}" type="revolute">
             <origin rpy="0 0 0" xyz="0.0 0.0 0.1475" />
-            <parent link="link_0" />
-            <child link="link_1" />
+            <parent link="${link_0_name}" />
+            <child link="${link_1_name}" />
             <axis xyz="0.0 0.0 1.0" />
             <limit
-                effort="${joint_limits['A1']['effort']}"
-                lower="${joint_limits['A1']['lower'] * PI / 180}"
-                upper="${joint_limits['A1']['upper'] * PI / 180}"
-                velocity="${joint_limits['A1']['velocity'] * PI / 180}" />
-            <dynamics damping="${joint_damping}" friction="${joint_friction}" />
-        </joint>
-        <link name="link_1">
+                effort="${joint_limits[joint_a1_name]['effort']}"
+                lower="${joint_limits[joint_a1_name]['lower'] * PI / 180}"
+                upper="${joint_limits[joint_a1_name]['upper'] * PI / 180}"
+                velocity="${joint_limits[joint_a1_name]['velocity'] * PI / 180}" />
+            <dynamics damping="${joint_damping}" friction="${joint_friction}" />
+        </joint>
+        <link name="${link_1_name}">
             <inertial>
                 <origin rpy="0 0 0" xyz="0.0 -0.034819 0.123299" />
@@ -74,17 +113,17 @@
             </collision>
         </link>
-        <joint name="A2" type="revolute">
+        <joint name="${joint_a2_name}" type="revolute">
             <origin rpy="0 0 0" xyz="0.0 -0.0105 0.1925" />
-            <parent link="link_1" />
-            <child link="link_2" />
+            <parent link="${link_1_name}" />
+            <child link="${link_2_name}" />
             <axis xyz="0.0 1.0 0.0" />
             <limit
-                effort="${joint_limits['A2']['effort']}"
-                lower="${joint_limits['A2']['lower'] * PI / 180}"
-                upper="${joint_limits['A2']['upper'] * PI / 180}"
-                velocity="${joint_limits['A2']['velocity'] * PI / 180}" />
-            <dynamics damping="${joint_damping}" friction="${joint_friction}" />
-        </joint>
-        <link name="link_2">
+                effort="${joint_limits[joint_a2_name]['effort']}"
+                lower="${joint_limits[joint_a2_name]['lower'] * PI / 180}"
+                upper="${joint_limits[joint_a2_name]['upper'] * PI / 180}"
+                velocity="${joint_limits[joint_a2_name]['velocity'] * PI / 180}" />
+            <dynamics damping="${joint_damping}" friction="${joint_friction}" />
+        </joint>
+        <link name="${link_2_name}">
             <inertial>
                 <origin rpy="0 0 0" xyz="0.0 0.039793 0.086944" />
@@ -106,17 +145,17 @@
             </collision>
         </link>
-        <joint name="A3" type="revolute">
+        <joint name="${joint_a3_name}" type="revolute">
             <origin rpy="0 0 0" xyz="0.0 0.0105 0.2075" />
-            <parent link="link_2" />
-            <child link="link_3" />
+            <parent link="${link_2_name}" />
+            <child link="${link_3_name}" />
             <axis xyz="0.0 0.0 1.0" />
             <limit
-                effort="${joint_limits['A3']['effort']}"
-                lower="${joint_limits['A3']['lower'] * PI / 180}"
-                upper="${joint_limits['A3']['upper'] * PI / 180}"
-                velocity="${joint_limits['A3']['velocity'] * PI / 180}" />
-            <dynamics damping="${joint_damping}" friction="${joint_friction}" />
-        </joint>
-        <link name="link_3">
+                effort="${joint_limits[joint_a3_name]['effort']}"
+                lower="${joint_limits[joint_a3_name]['lower'] * PI / 180}"
+                upper="${joint_limits[joint_a3_name]['upper'] * PI / 180}"
+                velocity="${joint_limits[joint_a3_name]['velocity'] * PI / 180}" />
+            <dynamics damping="${joint_damping}" friction="${joint_friction}" />
+        </joint>
+        <link name="${link_3_name}">
             <inertial>
                 <origin rpy="0 0 0" xyz="0.0 0.034819 0.123299" />
@@ -138,17 +177,17 @@
             </collision>
         </link>
-        <joint name="A4" type="revolute">
+        <joint name="${joint_a4_name}" type="revolute">
             <origin rpy="0 0 0" xyz="0.0 0.0105 0.1925" />
-            <parent link="link_3" />
-            <child link="link_4" />
+            <parent link="${link_3_name}" />
+            <child link="${link_4_name}" />
             <axis xyz="0.0 -1.0 0.0" />
             <limit
-                effort="${joint_limits['A4']['effort']}"
-                lower="${joint_limits['A4']['lower'] * PI / 180}"
-                upper="${joint_limits['A4']['upper'] * PI / 180}"
-                velocity="${joint_limits['A4']['velocity'] * PI / 180}" />
-            <dynamics damping="${joint_damping}" friction="${joint_friction}" />
-        </joint>
-        <link name="link_4">
+                effort="${joint_limits[joint_a4_name]['effort']}"
+                lower="${joint_limits[joint_a4_name]['lower'] * PI / 180}"
+                upper="${joint_limits[joint_a4_name]['upper'] * PI / 180}"
+                velocity="${joint_limits[joint_a4_name]['velocity'] * PI / 180}" />
+            <dynamics damping="${joint_damping}" friction="${joint_friction}" />
+        </joint>
+        <link name="${link_4_name}">
             <inertial>
                 <origin rpy="0 0 0" xyz="0.0 -0.039793 0.086944" />
@@ -170,17 +209,17 @@
             </collision>
         </link>
-        <joint name="A5" type="revolute">
+        <joint name="${joint_a5_name}" type="revolute">
             <origin rpy="0 0 0" xyz="0.0 -0.0105 0.2075" />
-            <parent link="link_4" />
-            <child link="link_5" />
+            <parent link="${link_4_name}" />
+            <child link="${link_5_name}" />
             <axis xyz="0.0 0.0 1.0" />
             <limit
-                effort="${joint_limits['A5']['effort']}"
-                lower="${joint_limits['A5']['lower'] * PI / 180}"
-                upper="${joint_limits['A5']['upper'] * PI / 180}"
-                velocity="${joint_limits['A5']['velocity'] * PI / 180}" />
-            <dynamics damping="${joint_damping}" friction="${joint_friction}" />
-        </joint>
-        <link name="link_5">
+                effort="${joint_limits[joint_a5_name]['effort']}"
+                lower="${joint_limits[joint_a5_name]['lower'] * PI / 180}"
+                upper="${joint_limits[joint_a5_name]['upper'] * PI / 180}"
+                velocity="${joint_limits[joint_a5_name]['velocity'] * PI / 180}" />
+            <dynamics damping="${joint_damping}" friction="${joint_friction}" />
+        </joint>
+        <link name="${link_5_name}">
             <inertial>
                 <origin rpy="0 0 0" xyz="0.0 -0.029824 0.076267" />
@@ -202,17 +241,17 @@
             </collision>
         </link>
-        <joint name="A6" type="revolute">
+        <joint name="${joint_a6_name}" type="revolute">
             <origin rpy="0 0 0" xyz="0.0 -0.0707 0.1925" />
-            <parent link="link_5" />
-            <child link="link_6" />
+            <parent link="${link_5_name}" />
+            <child link="${link_6_name}" />
             <axis xyz="0.0 1.0 0.0" />
             <limit
-                effort="${joint_limits['A6']['effort']}"
-                lower="${joint_limits['A6']['lower'] * PI / 180}"
-                upper="${joint_limits['A6']['upper'] * PI / 180}"
-                velocity="${joint_limits['A6']['velocity'] * PI / 180}" />
-            <dynamics damping="${joint_damping}" friction="${joint_friction}" />
-        </joint>
-        <link name="link_6">
+                effort="${joint_limits[joint_a6_name]['effort']}"
+                lower="${joint_limits[joint_a6_name]['lower'] * PI / 180}"
+                upper="${joint_limits[joint_a6_name]['upper'] * PI / 180}"
+                velocity="${joint_limits[joint_a6_name]['velocity'] * PI / 180}" />
+            <dynamics damping="${joint_damping}" friction="${joint_friction}" />
+        </joint>
+        <link name="${link_6_name}">
             <inertial>
                 <origin rpy="0 0 0" xyz="0.0 0.07102 0.00495" />
@@ -234,21 +273,22 @@
             </collision>
         </link>
-        <joint name="A7" type="revolute">
+        <joint name="${joint_a7_name}" type="revolute">
             <origin rpy="0 0 0" xyz="0.0 0.0707 0.091" />
-            <parent link="link_6" />
-            <child link="link_7" />
+            <parent link="${link_6_name}" />
+            <child link="${link_7_name}" />
             <axis xyz="0.0 0.0 1.0" />
             <limit
-                effort="${joint_limits['A7']['effort']}"
-                lower="${joint_limits['A7']['lower'] * PI / 180}"
-                upper="${joint_limits['A7']['upper'] * PI / 180}"
-                velocity="${joint_limits['A7']['velocity'] * PI / 180}" />
-            <dynamics damping="${joint_damping}" friction="${joint_friction}" />
-        </joint>
-        <link name="link_7">
+                effort="${joint_limits[joint_a7_name]['effort']}"
+                lower="${joint_limits[joint_a7_name]['lower'] * PI / 180}"
+                upper="${joint_limits[joint_a7_name]['upper'] * PI / 180}"
+                velocity="${joint_limits[joint_a7_name]['velocity'] * PI / 180}" />
+            <dynamics damping="${joint_damping}" friction="${joint_friction}" />
+        </joint>
+        <link name="${link_7_name}">
             <inertial>
                 <origin rpy="0 0 0" xyz="3.0000e-06 -2.0000e-06 1.3782e-02" />
                 <mass value="0.259474" />
-                <inertia ixx="0.000171" ixy="0.0" ixz="0.0" iyy="0.000171" iyz="0.0" izz="0.000299" />
+                <inertia ixx="0.000171" ixy="0.0" ixz="0.0" iyy="0.000171" iyz="0.0"
+                    izz="0.000299" />
             </inertial>
             <visual>
@@ -265,11 +305,4 @@
             </collision>
         </link>
-        <!-- <joint name="joint_ee" type="fixed">
-            <parent link="link_7" />
-            <child link="link_ee" />
-            <origin xyz="0 0 0.035" rpy="0 0 0" />
-        </joint>
-        <link name="link_ee">
-        </link> -->
     </xacro:macro>
 </robot>

File: src/lbr_fri_ros2_stack/lbr_description/urdf/kuka_blue/kuka_blue.xacro (robot description, xacro)
@@ -3,5 +3,5 @@
 <robot name="iiwa7" xmlns:xacro="http://www.ros.org/wiki/xacro">
     <!-- include the lbr iiwa macro -->
-    <xacro:include filename="$(find lbr_description)/urdf/iiwa7/iiwa7_description_mod.xacro" />
+    <xacro:include filename="$(find lbr_description)/urdf/iiwa7/iiwa7_description.xacro" />
     <!-- <xacro:include filename="$(find robotiq_description)/urdf/robotiq_2f_85_macro.urdf.xacro" /> -->
     <xacro:arg name="sim" default="true" />
@@ -26,5 +26,6 @@
         sim="$(arg sim)"
         system_parameters_path="$(arg system_parameters_path)"
-        controllers_path="$(arg controllers_path)" />
+        controllers_path="$(arg controllers_path)"
+        prefix_model_names="true" />
     <!-- End Effector -->
     <link name="${robot_prefix}_link_ee">

File: src/lbr_fri_ros2_stack/lbr_moveit_config/dual_iiwa7_moveit_config/config/dual_iiwa7.urdf.xacro (robot description, xacro)
@@ -2,6 +2,6 @@
 <robot xmlns:xacro="http://www.ros.org/wiki/xacro" name="dual_iiwa7">
     <xacro:arg name="initial_positions_file" default="initial_positions.yaml" />
-    <!-- Import dual_iiwa7 urdf file -->
-    <xacro:include filename="$(find lbr_description)/urdf/dual_iiwa7/dual_iiwa7_mod.urdf" />
+    <!-- Import the dual-arm scene xacro -->
+    <xacro:include filename="$(find lbr_description)/urdf/dual_iiwa7/dual_iiwa7.xacro" />
     <!-- Import control_xacro -->
     <xacro:include filename="dual_iiwa7.ros2_control.xacro" />
