Commit message: larege refractor.

File: src/lbr_fri_ros2_stack/lbr_description/urdf/iiwa14/iiwa14.xacro (robot description, xacro)
@@ -26,3 +26,9 @@
         system_parameters_path="$(arg system_parameters_path)"
         controllers_path="$(arg controllers_path)" />
+    <joint name="joint_ee" type="fixed">
+        <parent link="link_7" />
+        <child link="link_ee" />
+        <origin xyz="0 0 0.035" rpy="0 0 0" />
+    </joint>
+    <link name="link_ee" />
 </robot>

File: src/lbr_fri_ros2_stack/lbr_description/urdf/iiwa14/iiwa14_description.xacro (robot description, xacro)
@@ -265,11 +265,4 @@
             </collision>
         </link>
-        <joint name="joint_ee" type="fixed">
-            <parent link="link_7" />
-            <child link="link_ee" />
-            <origin xyz="0 0 0.035" rpy="0 0 0" />
-        </joint>
-        <link name="link_ee">
-        </link>
     </xacro:macro>
 </robot>

File: src/lbr_fri_ros2_stack/lbr_description/urdf/iiwa7/iiwa7.xacro (robot description, xacro)
@@ -26,3 +26,9 @@
         system_parameters_path="$(arg system_parameters_path)"
         controllers_path="$(arg controllers_path)" />
+    <joint name="joint_ee" type="fixed">
+        <parent link="link_7" />
+        <child link="link_ee" />
+        <origin xyz="0 0 0.035" rpy="0 0 0" />
+    </joint>
+    <link name="link_ee" />
 </robot>

File: src/lbr_fri_ros2_stack/lbr_description/urdf/kuka_blue/kuka_blue.xacro (robot description, xacro)
@@ -4,6 +4,6 @@
     <!-- include the lbr iiwa macro -->
     <xacro:include filename="$(find lbr_description)/urdf/iiwa7/iiwa7_description.xacro" />
-    <!-- <xacro:include filename="$(find robotiq_description)/urdf/robotiq_2f_85_macro.urdf.xacro" /> -->
     <xacro:arg name="sim" default="true" />
+    <xacro:arg name="use_fake_hardware" default="true" />
     <xacro:arg
         name="system_parameters_path"
@@ -38,5 +38,5 @@
             <origin rpy="0 3.14 0" xyz="0.0 0.0 0.0" />
             <geometry>
-                <mesh filename="package://lbr_description/meshes/iiwa7/visual/aniket_gripper.dae" scale="0.001 0.001 0.001"/>
+                <mesh filename="package://lbr_description/meshes/end_effectors/aniket_gripper/visual/aniket_gripper.dae" scale="0.001 0.001 0.001" />
             </geometry>
         </visual>
@@ -44,21 +44,19 @@
             <origin rpy="0 3.14 0" xyz="0.0 0.0 0.0" />
             <geometry>
-                <mesh filename="package://lbr_description/meshes/iiwa7/collision/aniket_gripper.stl" scale="0.001 0.001 0.001"/>
+                <mesh filename="package://lbr_description/meshes/end_effectors/aniket_gripper/collision/aniket_gripper.stl" scale="0.001 0.001 0.001" />
             </geometry>
         </collision>
     </link>
     <joint name="${robot_prefix}_joint_ee" type="fixed">
-        <parent link="${robot_prefix}_link_7"/>
-        <child link="${robot_prefix}_link_ee"/>
-        <origin rpy="0 0 3.14" xyz="0 0 0.035"/>
+        <parent link="${robot_prefix}_link_7" />
+        <child link="${robot_prefix}_link_ee" />
+        <origin rpy="0 0 3.14" xyz="0 0 0.035" />
     </joint>
     <!-- TCP Link -->
-    <link name="${robot_prefix}_link_tcp"/>
+    <link name="${robot_prefix}_link_tcp" />
     <joint name="${robot_prefix}_joint_tcp" type="fixed">
-        <parent link="${robot_prefix}_link_ee"/>
-        <child link="${robot_prefix}_link_tcp"/>
-        <!-- <origin rpy="0 0 0" xyz="0.00051 -0.00012 0.23332"/> NO FORCE TOOL -->
-        <!-- <origin rpy="0 0 0" xyz="0.00243 0.0003 0.22498"/> -->
-        <origin rpy="0 0 0" xyz="0.0 0.0 0.33149"/>
+        <parent link="${robot_prefix}_link_ee" />
+        <child link="${robot_prefix}_link_tcp" />
+        <origin rpy="0 0 0" xyz="0.0 0.0 0.33149" />
     </joint>
 </robot>

File: src/lbr_fri_ros2_stack/lbr_description/urdf/kuka_green/kuka_green.xacro (robot description, xacro)
@@ -25,5 +25,5 @@
         <!-- <origin xyz="0 0 0" rpy="0 0 0"/> -->
         <!-- <origin xyz="0.8057409 0.6804944 -0.4295127" rpy="-0.0265684 0.0060622 -2.3834002"/> -->
-         <!--RSOriginal-->
+        <!--RSOriginal-->
         <!-- <origin xyz="0.7947345 0.694259 -0.4280015" rpy="-0.0227401 0.0105353 -2.3640002"/>   -->
         <!-- <origin xyz="0.7947345 0.694259 -0.4330015" rpy="-0.0227401 0.0105353 -2.3640002"/> -->
@@ -55,5 +55,5 @@
             <origin rpy="1.57 0 1.57" xyz="-0.0925 0 0" />
             <geometry>
-                <mesh filename="package://lbr_description/meshes/iiwa7/collision/robotiq_gripper.stl" scale="0.001 0.001 0.001"/>
+                <mesh filename="package://lbr_description/meshes/end_effectors/robotiq_gripper/visual/robotiq_gripper.dae" scale="0.001 0.001 0.001"/>
             </geometry>
         </visual>
@@ -61,14 +61,8 @@
             <origin rpy="1.57 0 1.57" xyz="-0.0925 0 0" />
             <geometry>
-                <mesh filename="package://lbr_description/meshes/iiwa7/collision/robotiq_gripper.stl" scale="0.001 0.001 0.001"/>
+                <mesh filename="package://lbr_description/meshes/end_effectors/robotiq_gripper/collision/robotiq_gripper.stl" scale="0.001 0.001 0.001"/>
             </geometry>
         </collision>
     </link>
-    <joint name="joint_ee" type="fixed">
-        <parent link="link_7"/>
-        <child link="link_ee"/>
-        <origin rpy="0 0 0" xyz="0 0 0.035"/>
-    </joint>
-    <link name="link_tcp"/>
     <joint name="joint_tcp" type="fixed">
         <parent link="link_ee"/>

File: src/lbr_fri_ros2_stack/lbr_description/urdf/med14/med14.xacro (robot description, xacro)
@@ -26,3 +26,9 @@
         system_parameters_path="$(arg system_parameters_path)"
         controllers_path="$(arg controllers_path)" />
+    <joint name="joint_ee" type="fixed">
+        <parent link="link_7" />
+        <child link="link_ee" />
+        <origin xyz="0 0 0.035" rpy="0 0 0" />
+    </joint>
+    <link name="link_ee" />
 </robot>

File: src/lbr_fri_ros2_stack/lbr_description/urdf/med14/med14_description.xacro (robot description, xacro)
@@ -265,11 +265,4 @@
             </collision>
         </link>
-        <joint name="joint_ee" type="fixed">
-            <parent link="link_7" />
-            <child link="link_ee" />
-            <origin xyz="0 0 0.035" rpy="0 0 0" />
-        </joint>
-        <link name="link_ee">
-        </link>
     </xacro:macro>
 </robot>

File: src/lbr_fri_ros2_stack/lbr_description/urdf/med7/med7.xacro (robot description, xacro)
@@ -26,3 +26,9 @@
         system_parameters_path="$(arg system_parameters_path)"
         controllers_path="$(arg controllers_path)" />
+    <joint name="joint_ee" type="fixed">
+        <parent link="link_7" />
+        <child link="link_ee" />
+        <origin xyz="0 0 0.035" rpy="0 0 0" />
+    </joint>
+    <link name="link_ee" />
 </robot>

File: src/lbr_fri_ros2_stack/lbr_description/urdf/med7/med7_description.xacro (robot description, xacro)
@@ -266,11 +266,4 @@
             </collision>
         </link>
-        <joint name="joint_ee" type="fixed">
-            <parent link="link_7" />
-            <child link="link_ee" />
-            <origin xyz="0 0 0.035" rpy="0 0 0" />
-        </joint>
-        <link name="link_ee">
-        </link>
     </xacro:macro>
 </robot>
